File: interface-board/_saved_interface-board.sch (KiCad schematic (older format))
At the start: 23 parts, among them J1 HECS, J10 AUX, J11 UART, J12 NTC1, J13 NTC1, J16 Conn_01x23, J2 CASEFAN1, J3 CASEFAN2, J6 HV+, J7 HV-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

Commit message: Added IMD LV connector
Parts:
- J10: symbol Connector_Generic:Conn_01x03 -> Connector_Generic:Conn_01x02
- J4: renamed from J?; footprint Connector_PinSocket_2.54mm:PinSocket_1x04_P2.54mm_Vertical -> Connector_Molex:Molex_KK-254_AE-6410-05A_1x05_P2.54mm_Vertical
Connections:
- net at J16.17 (Pin_17), JP2.1 (A): now also J10.2 (Pin_2); no longer J10.3 (Pin_3)
- net at J16.18 (Pin_18), JP3.1 (A): now also J10.1 (Pin_1); no longer J10.2 (Pin_2)
- net at J16.19 (Pin_19), JP4.1 (A): no longer J10.1 (Pin_1)
Changed lines of the file:
@@
 CAN-
 $Comp
-L Connector_Generic:Conn_01x03 J10
+L Connector_Generic:Conn_01x02 J10
 U 1 1 5C6BA890
 P 1750 7150
@@
 	1150 6750 1000 6750
 $Comp
-L Connector_Generic:Conn_01x05 J?
+L Connector_Generic:Conn_01x05 J4
 U 1 1 5C4FC040
 P 2750 5600
-F 0 "J?" H 2750 5300 50  0000 C CNN
+F 0 "J4" H 2750 5300 50  0000 C CNN
 F 1 "Bender-LV" V 2850 5550 50  0000 C CNN
-F 2 "Connector_PinSocket_2.54mm:PinSocket_1x04_P2.54mm_Vertical" H 2750 5600 50  0001 C CNN
+F 2 "Connector_Molex:Molex_KK-254_AE-6410-05A_1x05_P2.54mm_Vertical" H 2750 5600 50  0001 C CNN
 F 3 "~" H 2750 5600 50  0001 C CNN
 	1    2750 5600
@@
 $EndComp
 $Comp
-L power:GND #PWR?
+L power:GND #PWR0105
 U 1 1 5C509587
 P 3000 5700
-F 0 "#PWR?" H 3000 5450 50  0001 C CNN
+F 0 "#PWR0105" H 3000 5450 50  0001 C CNN
 F 1 "GND" V 3005 5572 50  0000 R CNN
 F 2 "" H 3000 5700 50  0001 C CNN
@@
 IMD_OK
 $Comp
-L power:+12V #PWR?
+L power:+12V #PWR0106
 U 1 1 5C51B056
 P 3000 5350
-F 0 "#PWR?" H 3000 5200 50  0001 C CNN
+F 0 "#PWR0106" H 3000 5200 50  0001 C CNN
 F 1 "+12V" H 3015 5523 50  0000 C CNN
 F 2 "" H 3000 5350 50  0001 C CNN
