File: interface-board/interface-board.sch (KiCad schematic (older format))
At the start: 82 parts

Commit message: Lots of interface-board layout done
Parts:
- removed C? (x4): C, Capacitor_THT:CP_Radial_D10.0mm_P5.00mm, symbol Device:C
- removed C? (x3): 0.68uF, Capacitor_THT:C_Rect_L18.0mm_W8.0mm_P15.00mm_FKS3_FKP3, symbol Device:C_Small
- removed C? (x5): 0.1uF, Capacitor_SMD:C_0603_1608Metric, symbol Device:C
- removed C? (x2): 10uF, Capacitor_SMD:C_0603_1608Metric, symbol Device:C
- removed C? (x2): 22pF, Capacitor_SMD:C_0603_1608Metric, symbol Device:C_Small
- removed C? (x3): 4700uF, Capacitor_THT:CP_Radial_D18.0mm_P7.50mm, symbol Device:C_Small
- removed D? (x4): D, Diode_THT:D_DO-41_SOD81_P10.16mm_Horizontal, symbol Device:D
- removed D? (x2): LED, LED_SMD:LED_0603_1608Metric, symbol Device:LED
- removed J?: RJ45, Connector_RJ:RJ45_Amphenol_54602-x08_Horizontal, symbol Connector:RJ45
- removed J?: Conn_02x03_Odd_Even, Connector_PinSocket_2.54mm:PinSocket_2x03_P2.54mm_Vertical, symbol Connector_Generic:Conn_02x03_Odd_Even
- removed L?: 1uH, CustomFootprints:Murata_DFE252012P_Inductor, symbol Device:L_Small
- removed L?: 0.15uH, CustomFootprints:PA2607, symbol Device:L_Small
- removed Q? (x4): Q_NMOS_GDS, Package_TO_SOT_SMD:TO-252-2, symbol Device:Q_NMOS_GDS
- removed R? (x9): R_US, Resistor_SMD:R_0603_1608Metric, symbol Device:R_US
- removed R? (x2): 1Ω, Resistor_SMD:R_2512_6332Metric, symbol Device:R_US
- removed R? (x5): 1k, Resistor_SMD:R_0603_1608Metric, symbol Device:R_US
- removed R?: 50k, Resistor_SMD:R_0603_1608Metric, symbol Device:R_US
- removed R? (x4): 10k, Resistor_SMD:R_0603_1608Metric, symbol Device:R_US
- removed RV?: 5k, Potentiometer_THT:Potentiometer_Piher_PT-15-V02_Vertical, symbol Device:R_POT_TRIM_US
- removed U?: DCM4623TD2J13D0T70, CustomFootprints:DCM4623TD2J13D0T70 w_landpattern, symbol interface-board-rescue:DCM4623TD2J13D0T70-AEROParts
- removed U?: R-78E5.0-0.5, Converter_DCDC:Converter_DCDC_RECOM_R-78E-0.5_THT, symbol Regulator_Switching:R-78E5.0-0.5
- removed U?: MCP2515-IST, Package_SO:TSSOP-20_4.4x6.5mm_P0.65mm, symbol interface-board-rescue:MCP2515-IST-Interface_CAN_LIN
- removed U?: MCP2551-I-SN, Package_SO:SOIC-8_3.9x4.9mm_P1.27mm, symbol Interface_CAN_LIN:MCP2551-I-SN
- removed U?: ATmega328P-AU, Package_QFP:TQFP-32_7x7mm_P0.8mm, symbol interface-board-rescue:ATmega328P-AU-MCU_Microchip_ATmega
- removed U?: LTV-827S, Package_DIP:SMDIP-8_W9.53mm, symbol Isolator:LTV-827S
- removed U? (x2): LTV-824, Package_DIP:DIP-8_W7.62mm, symbol Isolator:LTV-824
- removed Y?: 16MHz, Crystal:Crystal_HC49-U_Vertical, symbol Device:Crystal_Small
Connections:
- net labels removed: 12V_SAFETY_IN, 12V_UNMETERED, CTRL1, CTRL2, CTRL3, CTRL4, D10, DC_DC_EN, DC_DC_FAULT, EN, FANOUT0, FAULT, LED1, LED2, MISO, MOSI, RESET, SCK, TRIM, TRIM_EN
- wire segments 230 -> 72
Other:
- note added: "Global nets connected to this sheet: \nGND"
- note added: "Global nets connected to this sheet: \nGND, 12V"
- note added: "Global nets connected to this sheet: \nGND, 5V, SDA, SCL"
- note added: "Need to feed METERED 12V back in \nso that 5V power isn't being ignored"
- note added: "Shutdown loop in = 12V bus"
- note removed: "500V-rated\ncaps"
- note removed: "CAN Interface"
- note removed: "DC-DC"
- note removed: "HV->12V DC-DC"
- note removed: "HV-Interface"
- note removed: "HV\nDanger!"
- note removed: "ICSP"
- note removed: "Input Filtering"
- note removed: "May want to change value"
- note removed: "Move these caps to \nacross fan outputs?"
- note removed: "Output Filtering"
- note removed: "Power Connectors"
- note removed: "Pull high to disable"
- note removed: "Shutdown loop in is 12V bus"
- note removed: "Status LEDs"
- note removed: "Trim Control"
- note removed: "uC"

Commit message: interface-board getting there schematic-wise.
Parts:
- removed C?: 0.1uF, Capacitor_SMD:C_0603_1608Metric, symbol Device:C
- removed C?: 0.1uF, Capacitor_SMD:C_0603_1608Metric, symbol Device:C_Small
- removed R? (x2): 0.02, Resistor_SMD:R_2512_6332Metric, symbol Device:R_US
- removed R? (x2): 10, Resistor_SMD:R_0603_1608Metric, symbol Device:R_US
- removed U?: INA219, Package_SO:SOIC-8_3.9x4.9mm_P1.27mm, symbol interface-board-rescue:INA219-AEROParts
- added F?: 20A, symbol Device:Fuse
- added F?: 1A, symbol Device:Fuse
- added J?: TSMP, symbol Connector_Generic:Conn_01x02
- added J?: CASEFAN2, symbol Connector_Generic:Conn_01x02
- added J?: CASEFAN1, symbol Connector_Generic:Conn_01x02
- added J?: HECS, symbol Connector_Generic:Conn_01x05
- added J?: UART, symbol Connector_Generic:Conn_01x04
- added J?: RJ45, symbol Connector:RJ45
- added JP?: SolderJumper_2_Open, symbol Jumper:SolderJumper_2_Open
- added JP? (x2): SolderJumper_2_Bridged, symbol Jumper:SolderJumper_2_Bridged
Connections:
- net labels added: DC_DC_EN, DC_DC_FAULT, DC_DC_TRIM_EN, FANOUT0, UART_RX, UART_TX
- net labels removed: BATT_12V_UNMETERED, SCL, SDA
- wire segments 72 -> 108
Other:
- note added: "Global nets connected to this sheet: \nGND, 5V"
- note removed: "Main Current/Voltage Meter"
- note removed: "May want to \nchange value to\nbetter suit current\nrange."
- note removed: "Need to feed METERED 12V back in \nso that 5V power isn't being ignored"
- note removed: "Optional filter circuit. If not needed, \nresistors can be replaced with 0Ω, and \ncap can be desoldered."
- moved on the sheet: J?, JP?

Commit message: schematic almost done maybe hopefully
Parts:
- added F?: 2.5A, Fuse:Fuseholder_Cylinder-5x20mm_Schurter_0031_8201_Horizontal_Open, symbol Device:Fuse_Small
- added J? (x2): NTC1, symbol Connector_Generic:Conn_01x02
Connections:
- net labels added: TEMP_1, TEMP_2
- wire segments 108 -> 117
Other:
- note added: "2.5A fuses give some \nheadroom, maybe \nshould change to 2A."
- note removed: "2.5A fuse gives some \nheadroom, maybe \nshould change to 2A."
- moved on the sheet: J?

Commit message: more interface-board
Parts:
- added C? (x2): 470uF, Capacitor_THT:CP_Radial_D10.0mm_P5.00mm, symbol Device:C
Other:
- note added: "HV Danger!"
- moved on the sheet: J?
Changed lines of the file:
@@
 Comment4 ""
 $EndDescr
-Text Notes 2700 1000 2    50   ~ 0
+Text Notes 2750 1050 2    50   ~ 0
 2.5A fuses give some \nheadroom, maybe \nshould change to 2A.
 $Comp
 L Device:Fuse_Small F?
 U 1 1 5C49093C
-P 1950 1300
-F 0 "F?" H 1950 1485 50  0000 C CNN
-F 1 "2.5A" H 1950 1394 50  0000 C CNN
-F 2 "Fuse:Fuseholder_Cylinder-5x20mm_Schurter_0031_8201_Horizontal_Open" H 1950 1300 50  0001 C CNN
-F 3 "~" H 1950 1300 50  0001 C CNN
-	1    1950 1300
-	1    0    0    -1
-$EndComp
-Text Label 2250 1300 2    50   ~ 0
+P 2000 1350
+F 0 "F?" H 2000 1535 50  0000 C CNN
+F 1 "2.5A" H 2000 1444 50  0000 C CNN
+F 2 "Fuse:Fuseholder_Cylinder-5x20mm_Schurter_0031_8201_Horizontal_Open" H 2000 1350 50  0001 C CNN
+F 3 "~" H 2000 1350 50  0001 C CNN
+	1    2000 1350
+	1    0    0    -1
+$EndComp
+Text Label 2300 1350 2    50   ~ 0
 HV+
-Text Label 2250 1450 2    50   ~ 0
+Text Label 2300 1500 2    50   ~ 0
 HV-
 $Comp
@@
 L Connector_Generic:Conn_01x01 J?
 U 1 1 5C7C388D
-P 900 1450
-F 0 "J?" H 1050 1350 50  0000 C CNN
-F 1 "HV-" H 1150 1450 50  0000 C CNN
-F 2 "" H 900 1450 50  0001 C CNN
-F 3 "~" H 900 1450 50  0001 C CNN
-	1    900  1450
+P 950 1500
+F 0 "J?" H 1100 1400 50  0000 C CNN
+F 1 "HV-" H 1200 1500 50  0000 C CNN
+F 2 "" H 950 1500 50  0001 C CNN
+F 3 "~" H 950 1500 50  0001 C CNN
+	1    950  1500
 	-1   0    0    1
 $EndComp
@@
 L Connector_Generic:Conn_01x01 J?
 U 1 1 5C83C6D2
-P 900 1300
-F 0 "J?" H 900 1200 50  0000 C CNN
-F 1 "HV+" H 1150 1300 50  0000 C CNN
-F 2 "" H 900 1300 50  0001 C CNN
-F 3 "~" H 900 1300 50  0001 C CNN
-	1    900  1300
+P 950 1350
+F 0 "J?" H 950 1250 50  0000 C CNN
+F 1 "HV+" H 1200 1350 50  0000 C CNN
+F 2 "" H 950 1350 50  0001 C CNN
+F 3 "~" H 950 1350 50  0001 C CNN
+	1    950  1350
 	-1   0    0    1
 $EndComp
@@
 L Connector_Generic:Conn_01x02 J?
 U 1 1 5C871653
-P 1200 1050
-F 0 "J?" V 1166 862 50  0000 R CNN
-F 1 "IMD" V 1300 1050 50  0000 R CNN
-F 2 "" H 1200 1050 50  0001 C CNN
-F 3 "~" H 1200 1050 50  0001 C CNN
-	1    1200 1050
+P 1250 1100
+F 0 "J?" V 1216 912 50  0000 R CNN
+F 1 "IMD" V 1350 1100 50  0000 R CNN
+F 2 "" H 1250 1100 50  0001 C CNN
+F 3 "~" H 1250 1100 50  0001 C CNN
+	1    1250 1100
 	0    -1   -1   0
 $EndComp
 Wire Wire Line
-	1100 1300 1200 1300
-Wire Wire Line
-	1200 1250 1200 1300
-Wire Wire Line
-	1300 1250 1300 1450
-Wire Wire Line
-	1300 1450 1100 1450
-Wire Wire Line
-	2250 1300 2050 1300
-Connection ~ 1200 1300
+	1150 1350 1250 1350
+Wire Wire Line
+	1250 1300 1250 1350
+Wire Wire Line
+	1350 1300 1350 1500
+Wire Wire Line
+	1350 1500 1150 1500
+Wire Wire Line
+	2300 1350 2100 1350
+Connection ~ 1250 1350
 $Sheet
 S 4600 1250 1600 900
@@
 L Connector_Generic:Conn_01x02 J?
 U 1 1 5C4C2740
-P 1550 1050
-F 0 "J?" V 1516 862 50  0000 R CNN
-F 1 "TSMP" V 1650 1100 50  0000 R CNN
-F 2 "" H 1550 1050 50  0001 C CNN
-F 3 "~" H 1550 1050 50  0001 C CNN
-	1    1550 1050
+P 1600 1100
+F 0 "J?" V 1566 912 50  0000 R CNN
+F 1 "TSMP" V 1700 1150 50  0000 R CNN
+F 2 "" H 1600 1100 50  0001 C CNN
+F 3 "~" H 1600 1100 50  0001 C CNN
+	1    1600 1100
 	0    -1   -1   0
 $EndComp
 Wire Wire Line
-	1200 1300 1550 1300
-Wire Wire Line
-	1550 1250 1550 1300
-Connection ~ 1550 1300
-Wire Wire Line
-	1550 1300 1850 1300
-Wire Wire Line
-	1650 1250 1650 1450
-Wire Wire Line
-	1300 1450 1650 1450
-Connection ~ 1300 1450
+	1250 1350 1600 1350
+Wire Wire Line
+	1600 1300 1600 1350
+Connection ~ 1600 1350
+Wire Wire Line
+	1600 1350 1900 1350
+Wire Wire Line
+	1700 1300 1700 1500
+Wire Wire Line
+	1350 1500 1700 1500
+Connection ~ 1350 1500
 Wire Wire Line
 	4600 2650 4350 2650
@@
 L Connector:RJ45 J?
 U 1 1 5C565B8C
-P 3000 6150
-F 0 "J?" H 2670 6154 50  0000 R CNN
-F 1 "RJ45" H 2670 6245 50  0000 R CNN
-F 2 "" V 3000 6175 50  0001 C CNN
-F 3 "~" V 3000 6175 50  0001 C CNN
-	1    3000 6150
+P 3000 5550
+F 0 "J?" H 2670 5554 50  0000 R CNN
+F 1 "RJ45" H 2670 5645 50  0000 R CNN
+F 2 "" V 3000 5575 50  0001 C CNN
+F 3 "~" V 3000 5575 50  0001 C CNN
+	1    3000 5550
 	1    0    0    1
 $EndComp
@@
 L power:GND #PWR?
 U 1 1 5C569DF7
-P 3450 6700
-F 0 "#PWR?" H 3450 6450 50  0001 C CNN
-F 1 "GND" H 3455 6527 50  0000 C CNN
-F 2 "" H 3450 6700 50  0001 C CNN
-F 3 "" H 3450 6700 50  0001 C CNN
-	1    3450 6700
-	1    0    0    -1
-$EndComp
-Wire Wire Line
-	3450 6700 3450 6350
-Wire Wire Line
-	3450 6350 3400 6350
-Wire Wire Line
-	3450 6350 3450 6050
-Wire Wire Line
-	3450 6050 3400 6050
-Connection ~ 3450 6350
-Wire Wire Line
-	3400 5850 3700 5850
-Wire Wire Line
-	3400 5950 3700 5950
+P 3500 6100
+F 0 "#PWR?" H 3500 5850 50  0001 C CNN
+F 1 "GND" H 3505 5927 50  0000 C CNN
+F 2 "" H 3500 6100 50  0001 C CNN
+F 3 "" H 3500 6100 50  0001 C CNN
+	1    3500 6100
+	1    0    0    -1
+$EndComp
+Wire Wire Line
+	3500 6100 3500 5750
+Wire Wire Line
+	3500 5750 3500 5450
+Connection ~ 3500 5750
+Wire Wire Line
+	3400 5250 3700 5250
+Wire Wire Line
+	3400 5350 3700 5350
 Wire Wire Line
 	4600 1350 4300 1350
@@
 Text Label 4300 1450 0    50   ~ 0
 CAN-
-Text Label 3700 5850 2    50   ~ 0
+Text Label 3700 5250 2    50   ~ 0
 CAN+
-Text Label 3700 5950 2    50   ~ 0
+Text Label 3700 5350 2    50   ~ 0
 CAN-
 $Comp
 L Device:Fuse_Small F?
 U 1 1 5C584F9F
-P 1950 1450
-F 0 "F?" H 1950 1350 50  0000 C CNN
-F 1 "2.5A" H 1950 1250 50  0000 C CNN
-F 2 "Fuse:Fuseholder_Cylinder-5x20mm_Schurter_0031_8201_Horizontal_Open" H 1950 1450 50  0001 C CNN
-F 3 "~" H 1950 1450 50  0001 C CNN
-	1    1950 1450
-	1    0    0    -1
-$EndComp
-Wire Wire Line
-	1650 1450 1850 1450
-Connection ~ 1650 1450
-Wire Wire Line
-	2050 1450 2250 1450
+P 2000 1500
+F 0 "F?" H 2000 1400 50  0000 C CNN
+F 1 "2.5A" H 2000 1300 50  0000 C CNN
+F 2 "Fuse:Fuseholder_Cylinder-5x20mm_Schurter_0031_8201_Horizontal_Open" H 2000 1500 50  0001 C CNN
+F 3 "~" H 2000 1500 50  0001 C CNN
+	1    2000 1500
+	1    0    0    -1
+$EndComp
+Wire Wire Line
+	1700 1500 1900 1500
+Connection ~ 1700 1500
+Wire Wire Line
+	2100 1500 2300 1500
 Text Label 6500 1900 2    50   ~ 0
 TEMP_1
@@
 Text Label 2400 4700 2    50   ~ 0
 TEMP_2
+Wire Wire Line
+	3400 5450 3500 5450
+Wire Wire Line
+	3400 5750 3500 5750
+$Comp
+L Device:C C?
+U 1 1 5C62DA6B
+P 1950 6550
+AR Path="/5C62DA6B" Ref="C?"  Part="1"
+AR Path="/5C5EE841/5C62DA6B" Ref="C?"  Part="1"
+F 0 "C?" H 2065 6596 50  0000 L CNN
+F 1 "470uF" H 2065 6505 50  0000 L CNN
+F 2 "Capacitor_THT:CP_Radial_D10.0mm_P5.00mm" H 1988 6400 50  0001 C CNN
+F 3 "~" H 1950 6550 50  0001 C CNN
+	1    1950 6550
+	1    0    0    -1
+$EndComp
+$Comp
+L power:GND #PWR?
+U 1 1 5C62DA87
+P 1950 6700
+AR Path="/5C62DA87" Ref="#PWR?"  Part="1"
+AR Path="/5C5EE841/5C62DA87" Ref="#PWR?"  Part="1"
+F 0 "#PWR?" H 1950 6450 50  0001 C CNN
+F 1 "GND" H 1955 6527 50  0000 C CNN
+F 2 "" H 1950 6700 50  0001 C CNN
+F 3 "" H 1950 6700 50  0001 C CNN
+	1    1950 6700
+	1    0    0    -1
+$EndComp
+$Comp
+L power:+12V #PWR?
+U 1 1 5C62DA9F
+P 1950 6400
+AR Path="/5C62DA9F" Ref="#PWR?"  Part="1"
+AR Path="/5C5EE841/5C62DA9F" Ref="#PWR?"  Part="1"
+F 0 "#PWR?" H 1950 6250 50  0001 C CNN
+F 1 "+12V" H 1965 6573 50  0000 C CNN
+F 2 "" H 1950 6400 50  0001 C CNN
+F 3 "" H 1950 6400 50  0001 C CNN
+	1    1950 6400
+	1    0    0    -1
+$EndComp
+$Comp
+L power:+12V #PWR?
+U 1 1 5C62DAA5
+P 2400 6400
+AR Path="/5C62DAA5" Ref="#PWR?"  Part="1"
+AR Path="/5C5EE841/5C62DAA5" Ref="#PWR?"  Part="1"
+F 0 "#PWR?" H 2400 6250 50  0001 C CNN
+F 1 "+12V" H 2415 6573 50  0000 C CNN
+F 2 "" H 2400 6400 50  0001 C CNN
+F 3 "" H 2400 6400 50  0001 C CNN
+	1    2400 6400
+	1    0    0    -1
+$EndComp
+$Comp
+L power:GND #PWR?
+U 1 1 5C62DA8D
+P 2400 6700
+AR Path="/5C62DA8D" Ref="#PWR?"  Part="1"
+AR Path="/5C5EE841/5C62DA8D" Ref="#PWR?"  Part="1"
+F 0 "#PWR?" H 2400 6450 50  0001 C CNN
+F 1 "GND" H 2405 6527 50  0000 C CNN
+F 2 "" H 2400 6700 50  0001 C CNN
+F 3 "" H 2400 6700 50  0001 C CNN
+	1    2400 6700
+	1    0    0    -1
+$EndComp
+$Comp
+L Device:C C?
+U 1 1 5C62DA72
+P 2400 6550
+AR Path="/5C62DA72" Ref="C?"  Part="1"
+AR Path="/5C5EE841/5C62DA72" Ref="C?"  Part="1"
+F 0 "C?" H 2515 6596 50  0000 L CNN
+F 1 "470uF" H 2515 6505 50  0000 L CNN
+F 2 "Capacitor_THT:CP_Radial_D10.0mm_P5.00mm" H 2438 6400 50  0001 C CNN
+F 3 "~" H 2400 6550 50  0001 C CNN
+	1    2400 6550
+	1    0    0    -1
+$EndComp
+Wire Notes Line width 39 rgb(253, 0, 0)
+	550  550  2800 550
+Wire Notes Line width 39 rgb(255, 0, 0)
+	2800 550  2800 1800
+Wire Notes Line width 39 rgb(255, 0, 0)
+	2800 1800 550  1800
+Wire Notes Line width 39 rgb(255, 0, 0)
+	550  1800 550  550
+Text Notes 600  800  0    157  ~ 31
+HV Danger!
 $EndSCHEMATC

Commit message: Beginnings of board layout of interface-board
Parts:
- removed F? (x2): 2.5A, Fuse:Fuseholder_Cylinder-5x20mm_Schurter_0031_8201_Horizontal_Open, symbol Device:Fuse_Small
- F3, F4: renamed from F?; footprint (none) -> Fuse:Fuseholder_Cylinder-5x20mm_Schurter_0031_8201_Horizontal_Open
- J1: renamed from J?; footprint (none) -> Connector_Molex:Molex_KK-254_AE-6410-05A_1x05_P2.54mm_Vertical
- J10: renamed from J?; footprint (none) -> Connector_Wago:Wago_734-134_1x04_P3.50mm_Vertical
- J11: renamed from J?; footprint (none) -> Connector_PinSocket_2.54mm:PinSocket_1x04_P2.54mm_Vertical
- J12, J13: renamed from J?; footprint (none) -> Connector_Molex:Molex_KK-254_AE-6410-02A_1x02_P2.54mm_Vertical
- J14: renamed from J?; footprint (none) -> Connector_RJ:RJ45_Amphenol_54602-x08_Horizontal
- J2, J3: renamed from J?; footprint (none) -> Connector:FanPinHeader_1x03_P2.54mm_Vertical
- J4: renamed from J?; footprint (none) -> Connector_JST:JST_ZE_B08B-ZESK-1D_1x08_P1.50mm_Vertical
- J5: renamed from J?; footprint (none) -> CustomFootprints:AMPSEAL 776266-1 14-PIN
- J6, J7: renamed from J?; footprint (none) -> MountingHole:MountingHole_4.3mm_M4_Pad_Via
- J8, J9: renamed from J?; footprint (none) -> Connector_Phoenix_MC_HighVoltage:PhoenixContact_MCV_1,5_2-G-5.08_1x02_P5.08mm_Vertical
- JP1, JP2, JP3, JP4, JP5: renamed from JP?; footprint (none) -> Jumper:SolderJumper-2_P1.3mm_Open_RoundedPad1.0x1.5mm
- JP6, JP7: renamed from JP?; footprint (none) -> Jumper:SolderJumper-2_P1.3mm_Bridged_RoundedPad1.0x1.5mm
- gave numbers to parts that had none: 2
Connections:
- wire segments 117 -> 115
Other:
- note added: "Fuses?"
- note removed: "2.5A fuses give some \nheadroom, maybe \nshould change to 2A."

Commit message: Updated main connector and pinout
Parts:
- removed J4: AMPSEAL_PWR, Connector_JST:JST_ZE_B08B-ZESK-1D_1x08_P1.50mm_Vertical, symbol Connector_Generic:Conn_01x08
- removed J5: AMPSEAL_MAIN, CustomFootprints:AMPSEAL 776266-1 14-PIN, symbol Connector_Generic:Conn_01x14
- removed JP1: Jumper, Jumper:SolderJumper-2_P1.3mm_Open_RoundedPad1.0x1.5mm, symbol Jumper:SolderJumper_2_Open
- added J16: Conn_01x23, 1-776087-1:TE_1-776087-1, symbol Connector_Generic:Conn_01x23
- J10: symbol Connector_Generic:Conn_01x04 -> Connector_Generic:Conn_01x03
Connections:
- net +12V: now also J16.14 (Pin_14), J16.6 (Pin_6)
- net +5V: now also J16.23 (Pin_23)
- net CAN+: now also J16.11 (Pin_11)
- net CAN-: now also J16.12 (Pin_12)
- net FANOUT1: now also J16.8 (Pin_8)
- net FANOUT2: now also J16.15 (Pin_15)
- net FANOUT3: now also J16.7 (Pin_7)
- net GND: now also J16.13 (Pin_13), J16.3 (Pin_3), J16.4 (Pin_4), J16.5 (Pin_5)
- net IMD_AN1: now also J16.20 (Pin_20)
- net IMD_AN2: now also J16.21 (Pin_21)
- net IMD_AN3: now also J16.22 (Pin_22)
- net SHDN_LOOP_OUT: now also J16.1 (Pin_1), J16.10 (Pin_10), J16.16 (Pin_16), J16.2 (Pin_2), J16.9 (Pin_9)
- net at J10.3 (Pin_3), JP2.1 (A): now also J16.17 (Pin_17)
- net at J10.2 (Pin_2), JP3.1 (A): now also J16.18 (Pin_18)
- net at J10.1 (Pin_1), JP4.1 (A): now also J16.19 (Pin_19)
Other:
- note removed: "Shutdown loop in = 12V bus"
- moved on the sheet: C1, C2, JP2, JP3, JP4

Commit message: Added IMD LV connector
Parts:
- removed J14: RJ45, Connector_RJ:RJ45_Amphenol_54602-x08_Horizontal, symbol Connector:RJ45
- added J4: Bender-LV, Connector_Molex:Molex_KK-254_AE-6410-05A_1x05_P2.54mm_Vertical, symbol Connector_Generic:Conn_01x05
Connections:
- net +12V: now also J4.5 (Pin_5)
- net GND: now also J4.1 (Pin_1), J4.2 (Pin_2), J4.3 (Pin_3)
- new net IMD_OK: J4.4 (Pin_4)
Changed lines of the file:
@@
 Text Label 2450 3300 2    50   ~ 0
 UART_TX
-$Comp
-L Connector:RJ45 J14
-U 1 1 5C565B8C
-P 3000 5550
-F 0 "J14" H 2670 5554 50  0000 R CNN
-F 1 "RJ45" H 2670 5645 50  0000 R CNN
-F 2 "Connector_RJ:RJ45_Amphenol_54602-x08_Horizontal" V 3000 5575 50  0001 C CNN
-F 3 "~" V 3000 5575 50  0001 C CNN
-	1    3000 5550
-	1    0    0    1
-$EndComp
-$Comp
-L power:GND #PWR018
-U 1 1 5C569DF7
-P 3500 6100
-F 0 "#PWR018" H 3500 5850 50  0001 C CNN
-F 1 "GND" H 3505 5927 50  0000 C CNN
-F 2 "" H 3500 6100 50  0001 C CNN
-F 3 "" H 3500 6100 50  0001 C CNN
-	1    3500 6100
-	1    0    0    -1
-$EndComp
-Wire Wire Line
-	3500 6100 3500 5750
-Wire Wire Line
-	3500 5750 3500 5450
-Connection ~ 3500 5750
-Wire Wire Line
-	3400 5250 3700 5250
-Wire Wire Line
-	3400 5350 3700 5350
 Wire Wire Line
 	4600 1350 4300 1350
@@
 CAN+
 Text Label 4300 1450 0    50   ~ 0
-CAN-
-Text Label 3700 5250 2    50   ~ 0
-CAN+
-Text Label 3700 5350 2    50   ~ 0
 CAN-
 Connection ~ 1700 1500
@@
 Text Label 2400 4700 2    50   ~ 0
 TEMP_2
-Wire Wire Line
-	3400 5450 3500 5450
-Wire Wire Line
-	3400 5750 3500 5750
 $Comp
 L Device:C C1
@@
 Wire Wire Line
 	1150 6750 1000 6750
+$Comp
+L Connector_Generic:Conn_01x05 J4
+U 1 1 5C4FC040
+P 2750 5600
+F 0 "J4" H 2750 5300 50  0000 C CNN
+F 1 "Bender-LV" V 2850 5550 50  0000 C CNN
+F 2 "Connector_Molex:Molex_KK-254_AE-6410-05A_1x05_P2.54mm_Vertical" H 2750 5600 50  0001 C CNN
+F 3 "~" H 2750 5600 50  0001 C CNN
+	1    2750 5600
+	-1   0    0    1
+$EndComp
+$Comp
+L power:GND #PWR0105
+U 1 1 5C509587
+P 3000 5700
+F 0 "#PWR0105" H 3000 5450 50  0001 C CNN
+F 1 "GND" V 3005 5572 50  0000 R CNN
+F 2 "" H 3000 5700 50  0001 C CNN
+F 3 "" H 3000 5700 50  0001 C CNN
+	1    3000 5700
+	0    -1   -1   0
+$EndComp
+Wire Wire Line
+	2950 5600 2950 5700
+Connection ~ 2950 5700
+Wire Wire Line
+	2950 5700 2950 5800
+Wire Wire Line
+	2950 5700 3000 5700
+Wire Wire Line
+	2950 5500 3250 5500
+Text Label 3250 5500 2    50   ~ 0
+IMD_OK
+$Comp
+L power:+12V #PWR0106
+U 1 1 5C51B056
+P 3000 5350
+F 0 "#PWR0106" H 3000 5200 50  0001 C CNN
+F 1 "+12V" H 3015 5523 50  0000 C CNN
+F 2 "" H 3000 5350 50  0001 C CNN
+F 3 "" H 3000 5350 50  0001 C CNN
+	1    3000 5350
+	1    0    0    -1
+$EndComp
+Wire Wire Line
+	3000 5350 3000 5400
+Wire Wire Line
+	3000 5400 2950 5400
 $EndSCHEMATC
