File: interface-board/interface-board.sch (KiCad schematic (older format))
At the start: 23 parts, among them J1 HECS, J10 AUX, J11 UART, J12 NTC1, J13 NTC1, J16 Conn_01x23, J2 CASEFAN1, J3 CASEFAN2, J4 Bender-LV, J6 HV+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

Commit message: Fixed more shit
Parts:
- removed F3: 1A, Fuse:Fuseholder_Cylinder-5x20mm_Schurter_0031_8201_Horizontal_Open, symbol Device:Fuse
- removed JP4: Jumper, Jumper:SolderJumper-2_P1.3mm_Open_RoundedPad1.0x1.5mm, symbol Jumper:SolderJumper_2_Open
- J10: symbol Connector_Generic:Conn_01x03 -> Connector_Generic:Conn_01x02
Connections:
- net +5V: no longer J16.23 (Pin_23)
- net IMD_OK: now also J16.19 (Pin_19)
- net at J16.17 (Pin_17), JP2.1 (A): now also J10.2 (Pin_2); no longer J10.3 (Pin_3)
- net at J16.18 (Pin_18), JP3.1 (A): now also J10.1 (Pin_1); no longer J10.2 (Pin_2)
Changed lines of the file:
@@
 	1    0    0    -1
 $EndComp
-$Comp
-L Jumper:SolderJumper_2_Open JP4
-U 1 1 5C6A71E9
-P 2100 7250
-F 0 "JP4" H 2400 7250 50  0000 C CNN
-F 1 "Jumper" H 2650 7250 50  0000 C CNN
-F 2 "Jumper:SolderJumper-2_P1.3mm_Open_RoundedPad1.0x1.5mm" H 2100 7250 50  0001 C CNN
-F 3 "~" H 2100 7250 50  0001 C CNN
-	1    2100 7250
-	1    0    0    -1
-$EndComp
-Wire Wire Line
-	2300 7250 2250 7250
 Wire Wire Line
 	2250 7150 2300 7150
 Connection ~ 2300 7150
-Wire Wire Line
-	2300 7150 2300 7250
 Wire Wire Line
 	2250 7050 2300 7050
@@
 	1    0    0    -1
 $EndComp
-Wire Wire Line
-	2300 7300 2300 7250
-Connection ~ 2300 7250
 $Comp
 L power:GND #PWR08
@@
 CAN-
 $Comp
-L Connector_Generic:Conn_01x03 J10
+L Connector_Generic:Conn_01x02 J10
 U 1 1 5C6BA890
 P 1750 7150
@@
 Wire Wire Line
 	1000 7150 1950 7150
-Connection ~ 1950 7250
-Wire Wire Line
-	1000 7250 1950 7250
 Connection ~ 1950 7050
 Wire Wire Line
@@
 	1150 4100 1100 4100
 $Comp
-L Device:Fuse F3
-U 1 1 5C52E25F
-P 6400 2900
-F 0 "F3" V 6200 2900 50  0000 C CNN
-F 1 "1A" V 6300 2900 50  0000 C CNN
-F 2 "Fuse:Fuseholder_Cylinder-5x20mm_Schurter_0031_8201_Horizontal_Open" V 6330 2900 50  0001 C CNN
-F 3 "~" H 6400 2900 50  0001 C CNN
-	1    6400 2900
-	0    1    1    0
-$EndComp
-Wire Wire Line
-	6200 2900 6250 2900
-$Comp
 L power:+12V #PWR020
 U 1 1 5C530767
-P 6800 2900
-F 0 "#PWR020" H 6800 2750 50  0001 C CNN
-F 1 "+12V" H 6815 3073 50  0000 C CNN
-F 2 "" H 6800 2900 50  0001 C CNN
-F 3 "" H 6800 2900 50  0001 C CNN
-	1    6800 2900
-	1    0    0    -1
-$EndComp
-Wire Wire Line
-	6800 2900 6550 2900
+P 6500 2900
+F 0 "#PWR020" H 6500 2750 50  0001 C CNN
+F 1 "+12V" H 6515 3073 50  0000 C CNN
+F 2 "" H 6500 2900 50  0001 C CNN
+F 3 "" H 6500 2900 50  0001 C CNN
+	1    6500 2900
+	1    0    0    -1
+$EndComp
 $Comp
 L power:+5V #PWR019
@@
 	-1   0    0    -1
 $EndComp
-$Comp
-L power:+5V #PWR0101
-U 1 1 5C4E62B7
-P 1000 7650
-F 0 "#PWR0101" H 1000 7500 50  0001 C CNN
-F 1 "+5V" V 1000 7750 50  0000 L CNN
-F 2 "" H 1000 7650 50  0001 C CNN
-F 3 "" H 1000 7650 50  0001 C CNN
-	1    1000 7650
-	0    1    1    0
-$EndComp
 Text Label 1750 5450 2    50   ~ 0
 SHDN_LOOP_OUT
@@
 Wire Wire Line
 	3000 5400 2950 5400
+Wire Wire Line
+	2300 7150 2300 7300
+Wire Wire Line
+	1000 7250 1350 7250
+Text Label 1350 7250 2    50   ~ 0
+IMD_OK
+Wire Wire Line
+	6200 2900 6500 2900
 $EndSCHEMATC
