File: interface-board/interface-board.sch (KiCad schematic (older format))
At the start: 15 parts, among them J1 HECS, J11 UART, J12 NTC1, J13 NTC1, J16 Conn_01x23, J2 CASEFAN1, J3 CASEFAN2, J4 Bender-LV, J5 BLINKY, J6 HV+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

Commit message: dunno
Parts:
- added F?: 2A, CustomFootprints:Fuseholder_Cylinder-5x20mm_Schurter_0031_8201_Horizontal_Open_3d, symbol Device:Fuse
Changed lines of the file:
@@
 Wire Wire Line
 	1150 1400 1150 1500
+$Comp
+L Device:Fuse F?
+U 1 1 5C705837
+P 1400 2500
+F 0 "F?" V 1203 2500 50  0000 C CNN
+F 1 "2A" V 1294 2500 50  0000 C CNN
+F 2 "CustomFootprints:Fuseholder_Cylinder-5x20mm_Schurter_0031_8201_Horizontal_Open_3d" V 1330 2500 50  0001 C CNN
+F 3 "~" H 1400 2500 50  0001 C CNN
+	1    1400 2500
+	0    1    1    0
+$EndComp
 $EndSCHEMATC
