File: interface-board/interface-board.kicad_pcb (KiCad board)
At the start: 2 copper layers, 181.5 x 110 mm, 86 parts, among them J1 HECS, J10 AUX, J11 UART, J12 NTC1, J13 NTC1, J15 ICSP, J16 Conn_01x23, J2 CASEFAN1, J3 CASEFAN2, J4 Bender-LV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

Commit message: Interface-board largely routed
Parts:
- removed J10: AUX, Connector_Wago:Wago_734-134_1x04_P3.50mm_Vertical
- removed JP2, JP3: Jumper, Jumper:SolderJumper-2_P1.3mm_Open_RoundedPad1.0x1.5mm
- added C20: 2200uF, Capacitor_THT:CP_Radial_D18.0mm_P7.50mm, B.Cu at (0.83, -4.45)
- added C21: 2200uF, Capacitor_THT:CP_Radial_D18.0mm_P7.50mm, B.Cu at (0.00, -24.1)
- C12, C13, C14: value 4700uF -> 2200uF
- C2: value 470uF -> 2200uF; footprint Capacitor_THT:CP_Radial_D10.0mm_P5.00mm -> Capacitor_THT:CP_Radial_D18.0mm_P7.50mm
- J7: footprint MountingHole:MountingHole_4.3mm_M4_Pad_Via -> MountingHole:MountingHole_6.4mm_M6_Pad_Via
- L2, R1, R23: moved to B.Cu
- moved C2 80.1 mm to (33.9, -43.5), turned to 180 degrees
- moved C15 78.6 mm to (-15.7, -54.9), turned to 90 degrees
- moved U7 76.2 mm to (-20.8, -53.6), turned to 90 degrees
- moved C16 70.4 mm to (-12.6, -58.1), turned to 270 degrees
- moved C17 68.0 mm to (-15.7, -58.1), turned to 270 degrees
- moved J12 39.8 mm to (21.1, 15.9), turned to 270 degrees
- moved J13 36.3 mm to (21.1, 9.17), turned to 270 degrees
- moved R8 32.2 mm to (15.4, 12.3), turned to 90 degrees
- moved R7 31.4 mm to (15.4, 19.1), turned to 90 degrees
- moved C12 25.3 mm to (10.8, -40.0), turned to 90 degrees
- moved RN1 25.2 mm to (-10.5, -40.7), turned to 180 degrees
- moved D3 23.4 mm to (7.05, -60.0)
- moved J2 23.4 mm to (-6.92, -53.1)
- moved J3 23.4 mm to (0.70, -53.1)
- moved Q1 23.4 mm to (12.1, -53.7)
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Connections:
- C2 pad 1: +12V -> Net-(C12-Pad1)
- U3 pad 27: (no net) -> SDA
- U3 pad 28: (no net) -> SCL
- U8 pad 5: (no net) -> SCL
- U8 pad 6: (no net) -> SDA
Routing:
- net +5V: track 0.00 -> 404.5 mm, vias 0 -> 2
- net /DC_DC_TRIM_EN: track 0.00 -> 145.9 mm
- net /DC_DC_EN: track 0.00 -> 141.8 mm, vias 0 -> 2
- net /DC_DC_FAULT: track 2.44 -> 135.4 mm
- net /fanControl/FAN_CTRL_3: track 0.00 -> 96.0 mm, vias 0 -> 2
- net /fanControl/FAN_CTRL_1: track 0.00 -> 93.5 mm, vias 0 -> 2
- net /fanControl/FAN_CTRL_0: track 0.00 -> 91.3 mm, vias 0 -> 2
- net /fanControl/FAN_CTRL_2: track 0.00 -> 91.1 mm, vias 0 -> 2
- net +12V: track 0.00 -> 78.5 mm, vias 0 -> 1
- net /uC+CAN/MISO: track 0.00 -> 66.5 mm, vias 0 -> 2
- net /uC+CAN/MOSI: track 0.00 -> 62.3 mm, vias 0 -> 2
- net /uC+CAN/SCK: track 0.00 -> 59.7 mm, vias 0 -> 2
- net /TEMP_2: track 0.00 -> 45.5 mm
- net /TEMP_1: track 0.00 -> 42.2 mm
- net /uC+CAN/CAN_CS: track 0.00 -> 41.4 mm, vias 0 -> 2
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- added copper zone on B.Cu, net /DC->DC Converters/12V_OUT
- added copper zone on F.Cu, net /DC->DC Converters/12V_OUT
- added copper zone on F.Cu, net /FANOUT1
- added copper zone on F.Cu, net /FANOUT2
- added copper zone on F.Cu, net /FANOUT3
- added copper zone on B.Cu, net GND
- added copper zone on B.Cu, net Net-(C12-Pad1)
Other:
- net class Default: clearance 0.2 -> 0.1524; trace_width 0.25 -> 0.1524
- net class HV added: clearance 2.54, trace_width 1.27, via_dia 0.8, via_drill 0.4
- net class High Current 12V added: clearance 0.2032, trace_width 3.175, via_dia 0.8, via_drill 0.4
- rule pad_to_mask_clearance: 0.051 -> 0.0508
- rule trace_clearance: 0.2 -> 0.1524

Commit message: Fully routed, added blinky DC/DC, added silkscreen labels, bumped 5V traces up to 0.025"
Parts:
- removed the REF** at (39.8, -54.0)
- removed the REF** at (39.8, -4.00)
- added G***: LOGO, CustomFootprints:hvlightningsymbol, F.Cu at (219.3, 64.7)
- added G***: LOGO, CustomFootprints:hvlightningsymbol, F.Cu at (196.9, 136.6)
- added G***: LOGO, AERO_Logos:AERO_Logo_30x12mm, F.Cu at (131.7, 90.6)
- added G***: LOGO, CustomFootprints:hvlightningsymbol, B.Cu at (196.9, 137.1)
- added J5: BLINKY, Connector_Phoenix_MC_HighVoltage:PhoenixContact_MCV_1,5_2-G-5.08_1x02_P5.08mm_Vertical, B.Cu at (147.9, 134.0)
- added REF**: MountingHole_4.3mm_M4_Pad_Via, MountingHole:MountingHole_4.3mm_M4_Pad_Via, F.Cu at (154.7, 49.1)
- added REF**: MountingHole_4.3mm_M4_Pad_Via, MountingHole:MountingHole_4.3mm_M4_Pad_Via, F.Cu at (154.7, 99.1)
- added U10: EPM1510SJ, CustomFootprints:EPM1510SJ, B.Cu at (180.9, 122.0)
- J16: value Conn_01x23 -> AMPSEAL
- J7: footprint MountingHole:MountingHole_6.4mm_M6_Pad_Via -> MountingHole:MountingHole_4.3mm_M4_Pad_Via
- moved J7 157.6 mm to (174.7, 111.4)
- moved R18 154.4 mm to (191.3, 59.6)
- moved C1 154.4 mm to (85.3, 89.4)
- moved C10 154.4 mm to (227.2, 74.4)
- moved C11 154.4 mm to (227.2, 65.4)
- moved C12 154.4 mm to (125.7, 63.1)
- moved C13 154.4 mm to (139.1, 75.8)
- moved C14 154.4 mm to (134.6, 98.7)
- moved C15 154.4 mm to (99.3, 48.3)
- moved C16 154.4 mm to (102.3, 45.0)
- moved C17 154.4 mm to (99.3, 45.0)
- moved C18 154.4 mm to (106.9, 111.9)
- moved C19 154.4 mm to (112.0, 115.5)
- moved C2 154.4 mm to (148.8, 59.6)
- moved C20 154.4 mm to (115.8, 98.7)
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Connections:
- J16 pad 17: Net-(J10-Pad2) -> (no net)
- J16 pad 18: Net-(J10-Pad1) -> (no net)
Routing:
- net /HV+: track 50.4 -> 86.2 mm
- net /HV-: track 128.3 -> 153.8 mm
- net Net-(U1-Pad1): track 0.00 -> 21.8 mm, vias 0 -> 2
- net Net-(U1-Pad4): track 0.00 -> 16.9 mm, vias 0 -> 2
- net GND: track 41.2 -> 54.2 mm, vias 12 -> 11
- net Net-(J5-Pad2): track 0.00 -> 11.9 mm
- net Net-(J5-Pad1): track 0.00 -> 9.88 mm
- net Net-(C6-Pad1): track 0.00 -> 8.76 mm
- net Net-(C5-Pad1): track 0.00 -> 8.62 mm
- net Net-(C10-Pad1): track 55.8 -> 51.7 mm
- net Net-(R2-Pad1): track 0.00 -> 2.22 mm
- net Net-(R3-Pad2): track 0.00 -> 2.14 mm
- net /DC->DC Converters/HV+: track 12.7 -> 11.1 mm
- net /DC_DC_EN: track 141.8 -> 141.1 mm
- net /DC_DC_FAULT: track 135.4 -> 134.7 mm
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Other:
- board text added: "2 1 Thermistor"
- board text added: "2.5A"
- board text added: "DANGER: HIGH VOLTAGE"
- board text added: "Fans"
- board text added: "GLV TSV"
- board text added: "HECS"
- board text added: "ICSP"
- board text added: "IMD CTRL"
- board text added: "TSMP IMD"
- board text added: "TSV Indicator"
- board text added: "TSV Interface and GLV PD Board"
- board text added: "TSV+"
- board text added: "TSV-"
- board text added: "UART"
- board text added: "UVM AERO Willem Hillier 2/9/2019"

Commit message: Cleaned up 3d models
Parts:
- removed J9: TSMP, Connector_Phoenix_MC_HighVoltage:PhoenixContact_MCV_1,5_2-G-5.08_1x02_P5.08mm_Vertical
- J16: value AMPSEAL -> Conn_01x23
- J7: footprint MountingHole:MountingHole_4.3mm_M4_Pad_Via -> CustomFootprints:TE_MATE-N-LOK_1-770870-x_1x03_P4.14mm_Vertical; moved to B.Cu
- J8: value IMD -> HV+; footprint Connector_Phoenix_MC_HighVoltage:PhoenixContact_MCV_1,5_2-G-5.08_1x02_P5.08mm_Vertical -> CustomFootprints:TE_MATE-N-LOK_1-770870-x_1x03_P4.14mm_Vertical
- moved J7 11.0 mm to (179.6, 101.6), turned to 180 degrees
- moved J8 8.69 mm to (194.9, 112.4), turned to 180 degrees
- moved J6 4.08 mm to (213.3, 118.1)
- moved G*** 1.84 mm to (196.8, 138.4)
- moved G*** 1.33 mm to (196.8, 138.4)
Connections:
- J8 pad 2: /HV- -> /HV+
Routing:
- net /HV+: track 86.2 -> 79.3 mm
- net /HV-: track 153.8 -> 150.6 mm
Other:
- board text added: "+HV"
- board text added: "-HV"
- board text removed: "TSMP IMD"
