File: interface-board/file5C4BAF40.sch (KiCad schematic (older format))
At the start: 7 parts

Commit message: more interface-board
Other:
- moved on the sheet: C?, R?, U?
Changed lines of the file:
@@
 L interface-board-rescue:INA219-AEROParts U?
 U 1 1 5C4BB14F
-P 4000 3550
+P 7050 3500
 AR Path="/5C4BB14F" Ref="U?"  Part="1"
 AR Path="/5C4BAF41/5C4BB14F" Ref="U?"  Part="1"
-F 0 "U?" H 4025 4115 50  0000 C CNN
-F 1 "INA219" H 4025 4024 50  0000 C CNN
-F 2 "Package_SO:SOIC-8_3.9x4.9mm_P1.27mm" H 4100 3550 50  0001 C CNN
-F 3 "" H 4100 3550 50  0001 C CNN
-	1    4000 3550
+F 0 "U?" H 7075 4065 50  0000 C CNN
+F 1 "INA219" H 7075 3974 50  0000 C CNN
+F 2 "Package_SO:SOIC-8_3.9x4.9mm_P1.27mm" H 7150 3500 50  0001 C CNN
+F 3 "" H 7150 3500 50  0001 C CNN
+	1    7050 3500
 	-1   0    0    -1
 $EndComp
-Text Notes 2050 3450 0    50   ~ 0
+Text Notes 2950 3850 0    157  ~ 31
 May want to \nchange value to\nbetter suit current\nrange.
 $Comp
 L power:GND #PWR?
 U 1 1 5C4BB157
-P 4650 4000
+P 7700 3950
 AR Path="/5C4BB157" Ref="#PWR?"  Part="1"
 AR Path="/5C4BAF41/5C4BB157" Ref="#PWR?"  Part="1"
-F 0 "#PWR?" H 4650 3750 50  0001 C CNN
-F 1 "GND" H 4655 3827 50  0000 C CNN
-F 2 "" H 4650 4000 50  0001 C CNN
-F 3 "" H 4650 4000 50  0001 C CNN
-	1    4650 4000
+F 0 "#PWR?" H 7700 3700 50  0001 C CNN
+F 1 "GND" H 7705 3777 50  0000 C CNN
+F 2 "" H 7700 3950 50  0001 C CNN
+F 3 "" H 7700 3950 50  0001 C CNN
+	1    7700 3950
 	1    0    0    -1
 $EndComp
 Wire Wire Line
-	4650 4000 4650 3850
-Wire Wire Line
-	4400 3850 4650 3850
-Wire Wire Line
-	4400 3700 4650 3700
-Wire Wire Line
-	4650 3700 4650 3850
-Connection ~ 4650 3850
-Wire Wire Line
-	4400 3600 4650 3600
-Wire Wire Line
-	4650 3600 4650 3700
-Connection ~ 4650 3700
-Wire Notes Line
-	1950 2750 1950 4300
-Wire Notes Line
-	1950 4300 4850 4300
-Wire Notes Line
-	4850 4300 4850 2750
-Wire Notes Line
-	4850 2750 1950 2750
+	7700 3950 7700 3800
+Wire Wire Line
+	7450 3800 7700 3800
+Wire Wire Line
+	7450 3650 7700 3650
+Wire Wire Line
+	7700 3650 7700 3800
+Connection ~ 7700 3800
+Wire Wire Line
+	7450 3550 7700 3550
+Wire Wire Line
+	7700 3550 7700 3650
+Connection ~ 7700 3650
+Wire Notes Line
+	5000 2700 5000 4250
+Wire Notes Line
+	5000 4250 7900 4250
+Wire Notes Line
+	7900 4250 7900 2700
+Wire Notes Line
+	7900 2700 5000 2700
 $Comp
 L Device:R_US R?
 U 1 1 5C4BB169
-P 2800 3550
+P 5850 3500
 AR Path="/5C4BB169" Ref="R?"  Part="1"
 AR Path="/5C4BAF41/5C4BB169" Ref="R?"  Part="1"
-F 0 "R?" V 3150 3550 50  0000 C CNN
-F 1 "0.02" V 3050 3550 50  0000 C CNN
-F 2 "Resistor_SMD:R_2512_6332Metric" V 2840 3540 50  0001 C CNN
-F 3 "~" H 2800 3550 50  0001 C CNN
-	1    2800 3550
+F 0 "R?" V 6200 3500 50  0000 C CNN
+F 1 "0.02" V 6100 3500 50  0000 C CNN
+F 2 "Resistor_SMD:R_2512_6332Metric" V 5890 3490 50  0001 C CNN
+F 3 "~" H 5850 3500 50  0001 C CNN
+	1    5850 3500
 	-1   0    0    1
 $EndComp
 Wire Wire Line
-	2800 3950 2800 3700
-Text Notes 2000 2900 0    100  ~ 0
+	5850 3900 5850 3650
+Text Notes 5050 2850 0    100  ~ 0
 Main Current/Voltage Meter
 $Comp
 L Device:R_US R?
 U 1 1 5C4BB172
-P 3000 3400
+P 6050 3350
 AR Path="/5C4BB172" Ref="R?"  Part="1"
 AR Path="/5C4BAF41/5C4BB172" Ref="R?"  Part="1"
-F 0 "R?" V 2795 3400 50  0000 C CNN
-F 1 "10" V 2886 3400 50  0000 C CNN
-F 2 "Resistor_SMD:R_0603_1608Metric" V 3040 3390 50  0001 C CNN
-F 3 "~" H 3000 3400 50  0001 C CNN
-	1    3000 3400
+F 0 "R?" V 5845 3350 50  0000 C CNN
+F 1 "10" V 5936 3350 50  0000 C CNN
+F 2 "Resistor_SMD:R_0603_1608Metric" V 6090 3340 50  0001 C CNN
+F 3 "~" H 6050 3350 50  0001 C CNN
+	1    6050 3350
 	0    1    1    0
 $EndComp
@@
 L Device:R_US R?
 U 1 1 5C4BB179
-P 3000 3700
+P 6050 3650
 AR Path="/5C4BB179" Ref="R?"  Part="1"
 AR Path="/5C4BAF41/5C4BB179" Ref="R?"  Part="1"
-F 0 "R?" V 2795 3700 50  0000 C CNN
-F 1 "10" V 2886 3700 50  0000 C CNN
-F 2 "Resistor_SMD:R_0603_1608Metric" V 3040 3690 50  0001 C CNN
-F 3 "~" H 3000 3700 50  0001 C CNN
-	1    3000 3700
+F 0 "R?" V 5845 3650 50  0000 C CNN
+F 1 "10" V 5936 3650 50  0000 C CNN
+F 2 "Resistor_SMD:R_0603_1608Metric" V 6090 3640 50  0001 C CNN
+F 3 "~" H 6050 3650 50  0001 C CNN
+	1    6050 3650
 	0    1    1    0
 $EndComp
 Wire Wire Line
-	2850 3400 2800 3400
-Connection ~ 2800 3400
-Wire Wire Line
-	2850 3700 2800 3700
-Connection ~ 2800 3700
+	5900 3350 5850 3350
+Connection ~ 5850 3350
+Wire Wire Line
+	5900 3650 5850 3650
+Connection ~ 5850 3650
 $Comp
 L Device:C C?
 U 1 1 5C4BB184
-P 3300 3550
+P 6350 3500
 AR Path="/5C4BB184" Ref="C?"  Part="1"
 AR Path="/5C4BAF41/5C4BB184" Ref="C?"  Part="1"
-F 0 "C?" H 3415 3596 50  0000 L CNN
-F 1 "0.1uF" H 3400 3500 50  0000 L CNN
-F 2 "Capacitor_SMD:C_0603_1608Metric" H 3338 3400 50  0001 C CNN
-F 3 "~" H 3300 3550 50  0001 C CNN
-	1    3300 3550
+F 0 "C?" H 6465 3546 50  0000 L CNN
+F 1 "0.1uF" H 6450 3450 50  0000 L CNN
+F 2 "Capacitor_SMD:C_0603_1608Metric" H 6388 3350 50  0001 C CNN
+F 3 "~" H 6350 3500 50  0001 C CNN
+	1    6350 3500
 	1    0    0    -1
 $EndComp
 Wire Wire Line
-	3150 3400 3300 3400
-Wire Wire Line
-	3150 3700 3300 3700
-Connection ~ 3300 3400
-Connection ~ 3300 3700
-Wire Wire Line
-	3300 3400 3550 3400
-Wire Wire Line
-	3300 3700 3550 3700
-Text Label 4800 3400 2    50   ~ 0
+	6200 3350 6350 3350
+Wire Wire Line
+	6200 3650 6350 3650
+Connection ~ 6350 3350
+Connection ~ 6350 3650
+Wire Wire Line
+	6350 3350 6600 3350
+Wire Wire Line
+	6350 3650 6600 3650
+Text Label 7850 3350 2    50   ~ 0
 SCL
-Text Label 4800 3500 2    50   ~ 0
+Text Label 7850 3450 2    50   ~ 0
 SDA
 $Comp
 L power:+5V #PWR?
 U 1 1 5C4BB193
-P 4400 3000
+P 7450 2950
 AR Path="/5C4BB193" Ref="#PWR?"  Part="1"
 AR Path="/5C4BAF41/5C4BB193" Ref="#PWR?"  Part="1"
-F 0 "#PWR?" H 4400 2850 50  0001 C CNN
-F 1 "+5V" H 4415 3173 50  0000 C CNN
-F 2 "" H 4400 3000 50  0001 C CNN
-F 3 "" H 4400 3000 50  0001 C CNN
-	1    4400 3000
+F 0 "#PWR?" H 7450 2800 50  0001 C CNN
+F 1 "+5V" H 7465 3123 50  0000 C CNN
+F 2 "" H 7450 2950 50  0001 C CNN
+F 3 "" H 7450 2950 50  0001 C CNN
+	1    7450 2950
 	1    0    0    -1
 $EndComp
 Wire Wire Line
-	4400 3400 4800 3400
-Wire Wire Line
-	4400 3500 4800 3500
+	7450 3350 7850 3350
+Wire Wire Line
+	7450 3450 7850 3450
 $Comp
 L Device:R_US R?
 U 1 1 5C4BB19B
-P 2650 3550
+P 5700 3500
 AR Path="/5C4BB19B" Ref="R?"  Part="1"
 AR Path="/5C4BAF41/5C4BB19B" Ref="R?"  Part="1"
-F 0 "R?" V 3050 3550 50  0000 C CNN
-F 1 "0.02" V 2950 3550 50  0000 C CNN
-F 2 "Resistor_SMD:R_2512_6332Metric" V 2690 3540 50  0001 C CNN
-F 3 "~" H 2650 3550 50  0001 C CNN
-	1    2650 3550
+F 0 "R?" V 6100 3500 50  0000 C CNN
+F 1 "0.02" V 6000 3500 50  0000 C CNN
+F 2 "Resistor_SMD:R_2512_6332Metric" V 5740 3490 50  0001 C CNN
+F 3 "~" H 5700 3500 50  0001 C CNN
+	1    5700 3500
 	-1   0    0    1
 $EndComp
 Wire Wire Line
-	2650 3400 2800 3400
-Wire Wire Line
-	2650 3700 2800 3700
-Wire Notes Line
-	2900 3100 2900 3800
-Wire Notes Line
-	3400 3100 2900 3100
-Wire Notes Line
-	2900 3800 3400 3800
-Text Notes 2000 4250 0    50   ~ 0
+	5700 3350 5850 3350
+Wire Wire Line
+	5700 3650 5850 3650
+Wire Notes Line
+	5950 3050 5950 3750
+Wire Notes Line
+	6450 3050 5950 3050
+Wire Notes Line
+	5950 3750 6450 3750
+Text Notes 5050 4200 0    50   ~ 0
 Optional filter circuit. If not needed, \nresistors can be replaced with 0Ω, and \ncap can be desoldered.
 Wire Notes Line
-	3400 3100 3400 3800
-Wire Notes Line
-	3150 3800 3150 4000
+	6450 3050 6450 3750
+Wire Notes Line
+	6200 3750 6200 3950
 $Comp
 L Device:C_Small C?
 U 1 1 5C4BB1AA
-P 4500 3250
+P 7550 3200
 AR Path="/5C4BB1AA" Ref="C?"  Part="1"
 AR Path="/5C4BAF41/5C4BB1AA" Ref="C?"  Part="1"
-F 0 "C?" V 4300 3250 50  0000 C CNN
-F 1 "0.1uF" V 4400 3300 50  0000 C CNN
-F 2 "Capacitor_SMD:C_0603_1608Metric" H 4500 3250 50  0001 C CNN
-F 3 "~" H 4500 3250 50  0001 C CNN
-	1    4500 3250
+F 0 "C?" V 7350 3200 50  0000 C CNN
+F 1 "0.1uF" V 7450 3250 50  0000 C CNN
+F 2 "Capacitor_SMD:C_0603_1608Metric" H 7550 3200 50  0001 C CNN
+F 3 "~" H 7550 3200 50  0001 C CNN
+	1    7550 3200
 	0    1    1    0
 $EndComp
 Wire Wire Line
-	4400 3250 4400 3000
+	7450 3200 7450 2950
 $Comp
 L power:GND #PWR?
 U 1 1 5C4BB1B2
-P 4600 3250
+P 7650 3200
 AR Path="/5C4BB1B2" Ref="#PWR?"  Part="1"
 AR Path="/5C4BAF41/5C4BB1B2" Ref="#PWR?"  Part="1"
-F 0 "#PWR?" H 4600 3000 50  0001 C CNN
-F 1 "GND" V 4600 3200 50  0000 R CNN
-F 2 "" H 4600 3250 50  0001 C CNN
-F 3 "" H 4600 3250 50  0001 C CNN
-	1    4600 3250
+F 0 "#PWR?" H 7650 2950 50  0001 C CNN
+F 1 "GND" V 7650 3150 50  0000 R CNN
+F 2 "" H 7650 3200 50  0001 C CNN
+F 3 "" H 7650 3200 50  0001 C CNN
+	1    7650 3200
 	0    -1   -1   0
 $EndComp
-Connection ~ 4400 3250
-Wire Wire Line
-	2800 3050 1750 3050
-Wire Wire Line
-	2800 3050 2800 3400
-Wire Wire Line
-	2800 3950 1750 3950
-Text HLabel 1750 3050 0    50   Input ~ 0
+Connection ~ 7450 3200
+Wire Wire Line
+	5850 3000 4800 3000
+Wire Wire Line
+	5850 3000 5850 3350
+Wire Wire Line
+	5850 3900 4800 3900
+Text HLabel 4800 3000 0    50   Input ~ 0
 IN
-Text HLabel 1750 3950 0    50   Input ~ 0
+Text HLabel 4800 3900 0    50   Input ~ 0
 OUT
 $EndSCHEMATC

Commit message: Beginnings of board layout of interface-board
Parts:
- gave numbers to parts that had none: 7
Changed lines of the file:
@@
 P 7050 3500
 AR Path="/5C4BB14F" Ref="U?"  Part="1"
-AR Path="/5C4BAF41/5C4BB14F" Ref="U?"  Part="1"
-F 0 "U?" H 7075 4065 50  0000 C CNN
+AR Path="/5C4BAF41/5C4BB14F" Ref="U8"  Part="1"
+F 0 "U8" H 7075 4065 50  0000 C CNN
 F 1 "INA219" H 7075 3974 50  0000 C CNN
 F 2 "Package_SO:SOIC-8_3.9x4.9mm_P1.27mm" H 7150 3500 50  0001 C CNN
@@
 P 7700 3950
 AR Path="/5C4BB157" Ref="#PWR?"  Part="1"
-AR Path="/5C4BAF41/5C4BB157" Ref="#PWR?"  Part="1"
-F 0 "#PWR?" H 7700 3700 50  0001 C CNN
+AR Path="/5C4BAF41/5C4BB157" Ref="#PWR070"  Part="1"
+F 0 "#PWR070" H 7700 3700 50  0001 C CNN
 F 1 "GND" H 7705 3777 50  0000 C CNN
 F 2 "" H 7700 3950 50  0001 C CNN
@@
 P 5850 3500
 AR Path="/5C4BB169" Ref="R?"  Part="1"
-AR Path="/5C4BAF41/5C4BB169" Ref="R?"  Part="1"
-F 0 "R?" V 6200 3500 50  0000 C CNN
+AR Path="/5C4BAF41/5C4BB169" Ref="R25"  Part="1"
+F 0 "R25" V 6200 3500 50  0000 C CNN
 F 1 "0.02" V 6100 3500 50  0000 C CNN
 F 2 "Resistor_SMD:R_2512_6332Metric" V 5890 3490 50  0001 C CNN
@@
 P 6050 3350
 AR Path="/5C4BB172" Ref="R?"  Part="1"
-AR Path="/5C4BAF41/5C4BB172" Ref="R?"  Part="1"
-F 0 "R?" V 5845 3350 50  0000 C CNN
+AR Path="/5C4BAF41/5C4BB172" Ref="R26"  Part="1"
+F 0 "R26" V 5845 3350 50  0000 C CNN
 F 1 "10" V 5936 3350 50  0000 C CNN
 F 2 "Resistor_SMD:R_0603_1608Metric" V 6090 3340 50  0001 C CNN
@@
 P 6050 3650
 AR Path="/5C4BB179" Ref="R?"  Part="1"
-AR Path="/5C4BAF41/5C4BB179" Ref="R?"  Part="1"
-F 0 "R?" V 5845 3650 50  0000 C CNN
+AR Path="/5C4BAF41/5C4BB179" Ref="R27"  Part="1"
+F 0 "R27" V 5845 3650 50  0000 C CNN
 F 1 "10" V 5936 3650 50  0000 C CNN
 F 2 "Resistor_SMD:R_0603_1608Metric" V 6090 3640 50  0001 C CNN
@@
 P 6350 3500
 AR Path="/5C4BB184" Ref="C?"  Part="1"
-AR Path="/5C4BAF41/5C4BB184" Ref="C?"  Part="1"
-F 0 "C?" H 6465 3546 50  0000 L CNN
+AR Path="/5C4BAF41/5C4BB184" Ref="C18"  Part="1"
+F 0 "C18" H 6465 3546 50  0000 L CNN
 F 1 "0.1uF" H 6450 3450 50  0000 L CNN
 F 2 "Capacitor_SMD:C_0603_1608Metric" H 6388 3350 50  0001 C CNN
@@
 P 7450 2950
 AR Path="/5C4BB193" Ref="#PWR?"  Part="1"
-AR Path="/5C4BAF41/5C4BB193" Ref="#PWR?"  Part="1"
-F 0 "#PWR?" H 7450 2800 50  0001 C CNN
+AR Path="/5C4BAF41/5C4BB193" Ref="#PWR068"  Part="1"
+F 0 "#PWR068" H 7450 2800 50  0001 C CNN
 F 1 "+5V" H 7465 3123 50  0000 C CNN
 F 2 "" H 7450 2950 50  0001 C CNN
@@
 P 5700 3500
 AR Path="/5C4BB19B" Ref="R?"  Part="1"
-AR Path="/5C4BAF41/5C4BB19B" Ref="R?"  Part="1"
-F 0 "R?" V 6100 3500 50  0000 C CNN
+AR Path="/5C4BAF41/5C4BB19B" Ref="R24"  Part="1"
+F 0 "R24" V 6100 3500 50  0000 C CNN
 F 1 "0.02" V 6000 3500 50  0000 C CNN
 F 2 "Resistor_SMD:R_2512_6332Metric" V 5740 3490 50  0001 C CNN
@@
 P 7550 3200
 AR Path="/5C4BB1AA" Ref="C?"  Part="1"
-AR Path="/5C4BAF41/5C4BB1AA" Ref="C?"  Part="1"
-F 0 "C?" V 7350 3200 50  0000 C CNN
+AR Path="/5C4BAF41/5C4BB1AA" Ref="C19"  Part="1"
+F 0 "C19" V 7350 3200 50  0000 C CNN
 F 1 "0.1uF" V 7450 3250 50  0000 C CNN
 F 2 "Capacitor_SMD:C_0603_1608Metric" H 7550 3200 50  0001 C CNN
@@
 P 7650 3200
 AR Path="/5C4BB1B2" Ref="#PWR?"  Part="1"
-AR Path="/5C4BAF41/5C4BB1B2" Ref="#PWR?"  Part="1"
-F 0 "#PWR?" H 7650 2950 50  0001 C CNN
+AR Path="/5C4BAF41/5C4BB1B2" Ref="#PWR069"  Part="1"
+F 0 "#PWR069" H 7650 2950 50  0001 C CNN
 F 1 "GND" V 7650 3150 50  0000 R CNN
 F 2 "" H 7650 3200 50  0001 C CNN

Commit message: Interface-board largely routed
Changed lines of the file:
@@
 Wire Wire Line
 	6350 3650 6600 3650
-Text Label 7850 3350 2    50   ~ 0
-SCL
-Text Label 7850 3450 2    50   ~ 0
-SDA
 $Comp
 L power:+5V #PWR?
@@
 	1    0    0    -1
 $EndComp
-Wire Wire Line
-	7450 3350 7850 3350
-Wire Wire Line
-	7450 3450 7850 3450
 $Comp
 L Device:R_US R?
@@
 Text HLabel 4800 3900 0    50   Input ~ 0
 OUT
+Text HLabel 7650 3350 2    50   Input ~ 0
+SCL
+Text HLabel 7650 3450 2    50   Input ~ 0
+SDA
+Wire Wire Line
+	7650 3350 7450 3350
+Wire Wire Line
+	7450 3450 7650 3450
 $EndSCHEMATC
