File: interface-board/file5C5EE840.sch (KiCad schematic (older format))
At the start: 20 parts

Commit message: more interface-board
Parts:
- removed C? (x4): C, Capacitor_THT:CP_Radial_D10.0mm_P5.00mm, symbol Device:C
Other:
- note added: "Caps across fan outputs a good idea maybe?"
- note removed: "Move these caps to \nacross fan outputs?"
Changed lines of the file:
@@
 $EndComp
-$Comp
-L Device:C C?
-U 1 1 5C5EED44
-P 2050 3350
-AR Path="/5C5EED44" Ref="C?"  Part="1"
-AR Path="/5C5EE841/5C5EED44" Ref="C?"  Part="1"
-F 0 "C?" H 2165 3396 50  0000 L CNN
-F 1 "C" H 2165 3305 50  0000 L CNN
-F 2 "Capacitor_THT:CP_Radial_D10.0mm_P5.00mm" H 2088 3200 50  0001 C CNN
-F 3 "~" H 2050 3350 50  0001 C CNN
-	1    2050 3350
-	1    0    0    -1
-$EndComp
-$Comp
-L Device:C C?
-U 1 1 5C5EED4B
-P 2350 3350
-AR Path="/5C5EED4B" Ref="C?"  Part="1"
-AR Path="/5C5EE841/5C5EED4B" Ref="C?"  Part="1"
-F 0 "C?" H 2465 3396 50  0000 L CNN
-F 1 "C" H 2465 3305 50  0000 L CNN
-F 2 "Capacitor_THT:CP_Radial_D10.0mm_P5.00mm" H 2388 3200 50  0001 C CNN
-F 3 "~" H 2350 3350 50  0001 C CNN
-	1    2350 3350
-	1    0    0    -1
-$EndComp
-$Comp
-L Device:C C?
-U 1 1 5C5EED52
-P 2600 3350
-AR Path="/5C5EED52" Ref="C?"  Part="1"
-AR Path="/5C5EE841/5C5EED52" Ref="C?"  Part="1"
-F 0 "C?" H 2715 3396 50  0000 L CNN
-F 1 "C" H 2715 3305 50  0000 L CNN
-F 2 "Capacitor_THT:CP_Radial_D10.0mm_P5.00mm" H 2638 3200 50  0001 C CNN
-F 3 "~" H 2600 3350 50  0001 C CNN
-	1    2600 3350
-	1    0    0    -1
-$EndComp
-$Comp
-L Device:C C?
-U 1 1 5C5EED59
-P 2850 3350
-AR Path="/5C5EED59" Ref="C?"  Part="1"
-AR Path="/5C5EE841/5C5EED59" Ref="C?"  Part="1"
-F 0 "C?" H 2965 3396 50  0000 L CNN
-F 1 "C" H 2965 3305 50  0000 L CNN
-F 2 "Capacitor_THT:CP_Radial_D10.0mm_P5.00mm" H 2888 3200 50  0001 C CNN
-F 3 "~" H 2850 3350 50  0001 C CNN
-	1    2850 3350
-	1    0    0    -1
-$EndComp
-$Comp
-L power:GND #PWR?
-U 1 1 5C5EED60
-P 2050 3500
-AR Path="/5C5EED60" Ref="#PWR?"  Part="1"
-AR Path="/5C5EE841/5C5EED60" Ref="#PWR?"  Part="1"
-F 0 "#PWR?" H 2050 3250 50  0001 C CNN
-F 1 "GND" H 2055 3327 50  0000 C CNN
-F 2 "" H 2050 3500 50  0001 C CNN
-F 3 "" H 2050 3500 50  0001 C CNN
-	1    2050 3500
-	1    0    0    -1
-$EndComp
-$Comp
-L power:GND #PWR?
-U 1 1 5C5EED66
-P 2350 3500
-AR Path="/5C5EED66" Ref="#PWR?"  Part="1"
-AR Path="/5C5EE841/5C5EED66" Ref="#PWR?"  Part="1"
-F 0 "#PWR?" H 2350 3250 50  0001 C CNN
-F 1 "GND" H 2355 3327 50  0000 C CNN
-F 2 "" H 2350 3500 50  0001 C CNN
-F 3 "" H 2350 3500 50  0001 C CNN
-	1    2350 3500
-	1    0    0    -1
-$EndComp
-$Comp
-L power:GND #PWR?
-U 1 1 5C5EED6C
-P 2600 3500
-AR Path="/5C5EED6C" Ref="#PWR?"  Part="1"
-AR Path="/5C5EE841/5C5EED6C" Ref="#PWR?"  Part="1"
-F 0 "#PWR?" H 2600 3250 50  0001 C CNN
-F 1 "GND" H 2605 3327 50  0000 C CNN
-F 2 "" H 2600 3500 50  0001 C CNN
-F 3 "" H 2600 3500 50  0001 C CNN
-	1    2600 3500
-	1    0    0    -1
-$EndComp
-$Comp
-L power:GND #PWR?
-U 1 1 5C5EED72
-P 2850 3500
-AR Path="/5C5EED72" Ref="#PWR?"  Part="1"
-AR Path="/5C5EE841/5C5EED72" Ref="#PWR?"  Part="1"
-F 0 "#PWR?" H 2850 3250 50  0001 C CNN
-F 1 "GND" H 2855 3327 50  0000 C CNN
-F 2 "" H 2850 3500 50  0001 C CNN
-F 3 "" H 2850 3500 50  0001 C CNN
-	1    2850 3500
-	1    0    0    -1
-$EndComp
-$Comp
-L power:+12V #PWR?
-U 1 1 5C5EED78
-P 2050 3200
-AR Path="/5C5EED78" Ref="#PWR?"  Part="1"
-AR Path="/5C5EE841/5C5EED78" Ref="#PWR?"  Part="1"
-F 0 "#PWR?" H 2050 3050 50  0001 C CNN
-F 1 "+12V" H 2065 3373 50  0000 C CNN
-F 2 "" H 2050 3200 50  0001 C CNN
-F 3 "" H 2050 3200 50  0001 C CNN
-	1    2050 3200
-	1    0    0    -1
-$EndComp
-$Comp
-L power:+12V #PWR?
-U 1 1 5C5EED7E
-P 2350 3200
-AR Path="/5C5EED7E" Ref="#PWR?"  Part="1"
-AR Path="/5C5EE841/5C5EED7E" Ref="#PWR?"  Part="1"
-F 0 "#PWR?" H 2350 3050 50  0001 C CNN
-F 1 "+12V" H 2365 3373 50  0000 C CNN
-F 2 "" H 2350 3200 50  0001 C CNN
-F 3 "" H 2350 3200 50  0001 C CNN
-	1    2350 3200
-	1    0    0    -1
-$EndComp
-$Comp
-L power:+12V #PWR?
-U 1 1 5C5EED84
-P 2600 3200
-AR Path="/5C5EED84" Ref="#PWR?"  Part="1"
-AR Path="/5C5EE841/5C5EED84" Ref="#PWR?"  Part="1"
-F 0 "#PWR?" H 2600 3050 50  0001 C CNN
-F 1 "+12V" H 2615 3373 50  0000 C CNN
-F 2 "" H 2600 3200 50  0001 C CNN
-F 3 "" H 2600 3200 50  0001 C CNN
-	1    2600 3200
-	1    0    0    -1
-$EndComp
-$Comp
-L power:+12V #PWR?
-U 1 1 5C5EED8A
-P 2850 3200
-AR Path="/5C5EED8A" Ref="#PWR?"  Part="1"
-AR Path="/5C5EE841/5C5EED8A" Ref="#PWR?"  Part="1"
-F 0 "#PWR?" H 2850 3050 50  0001 C CNN
-F 1 "+12V" H 2865 3373 50  0000 C CNN
-F 2 "" H 2850 3200 50  0001 C CNN
-F 3 "" H 2850 3200 50  0001 C CNN
-	1    2850 3200
-	1    0    0    -1
-$EndComp
-Text Notes 2000 3900 0    50   ~ 0
-Move these caps to \nacross fan outputs?
 $Comp
 L power:GND #PWR?
@@
 	7450 4050 7400 4050
 Connection ~ 7400 4050
+Text Notes 2700 3300 0    157  ~ 31
+Caps across fan outputs a good idea maybe?
 $EndSCHEMATC

Commit message: Beginnings of board layout of interface-board
Parts:
- gave numbers to parts that had none: 16
Changed lines of the file:
@@
 P 4550 2500
 AR Path="/5C5EECB4" Ref="Q?"  Part="1"
-AR Path="/5C5EE841/5C5EECB4" Ref="Q?"  Part="1"
-F 0 "Q?" H 4800 2400 50  0000 C CNN
+AR Path="/5C5EE841/5C5EECB4" Ref="Q1"  Part="1"
+F 0 "Q1" H 4800 2400 50  0000 C CNN
 F 1 "Q_NMOS_GDS" H 5000 2550 50  0000 C CNN
 F 2 "Package_TO_SOT_SMD:TO-252-2" H 4750 2600 50  0001 C CNN
@@
 P 4300 2150
 AR Path="/5C5EECE9" Ref="D?"  Part="1"
-AR Path="/5C5EE841/5C5EECE9" Ref="D?"  Part="1"
-F 0 "D?" H 4300 2350 50  0000 C CNN
+AR Path="/5C5EE841/5C5EECE9" Ref="D3"  Part="1"
+F 0 "D3" H 4300 2350 50  0000 C CNN
 F 1 "1N4001" H 4300 2250 50  0000 C CNN
 F 2 "Diode_THT:D_DO-41_SOD81_P10.16mm_Horizontal" H 4300 2150 50  0001 C CNN
@@
 P 4100 2100
 AR Path="/5C5EECF0" Ref="#PWR?"  Part="1"
-AR Path="/5C5EE841/5C5EECF0" Ref="#PWR?"  Part="1"
-F 0 "#PWR?" H 4100 1950 50  0001 C CNN
+AR Path="/5C5EE841/5C5EECF0" Ref="#PWR045"  Part="1"
+F 0 "#PWR045" H 4100 1950 50  0001 C CNN
 F 1 "+12V" H 4115 2273 50  0000 C CNN
 F 2 "" H 4100 2100 50  0001 C CNN
@@
 P 5050 2650
 AR Path="/5C5EED0B" Ref="R?"  Part="1"
-AR Path="/5C5EE841/5C5EED0B" Ref="R?"  Part="1"
-F 0 "R?" H 4982 2604 50  0000 R CNN
+AR Path="/5C5EE841/5C5EED0B" Ref="R11"  Part="1"
+F 0 "R11" H 4982 2604 50  0000 R CNN
 F 1 "R_US" H 4982 2695 50  0000 R CNN
 F 2 "Resistor_SMD:R_0603_1608Metric" V 5090 2640 50  0001 C CNN
@@
 P 4900 2500
 AR Path="/5C5EED27" Ref="R?"  Part="1"
-AR Path="/5C5EE841/5C5EED27" Ref="R?"  Part="1"
-F 0 "R?" V 4800 2500 50  0000 C CNN
+AR Path="/5C5EE841/5C5EED27" Ref="R9"  Part="1"
+F 0 "R9" V 4800 2500 50  0000 C CNN
 F 1 "R_US" V 5000 2500 50  0000 C CNN
 F 2 "Resistor_SMD:R_0603_1608Metric" V 4940 2490 50  0001 C CNN
@@
 P 4450 2800
 AR Path="/5C5EEDC2" Ref="#PWR?"  Part="1"
-AR Path="/5C5EE841/5C5EEDC2" Ref="#PWR?"  Part="1"
-F 0 "#PWR?" H 4450 2550 50  0001 C CNN
+AR Path="/5C5EE841/5C5EEDC2" Ref="#PWR047"  Part="1"
+F 0 "#PWR047" H 4450 2550 50  0001 C CNN
 F 1 "GND" H 4455 2627 50  0000 C CNN
 F 2 "" H 4450 2800 50  0001 C CNN
@@
 P 5050 2800
 AR Path="/5C5F2488" Ref="#PWR?"  Part="1"
-AR Path="/5C5EE841/5C5F2488" Ref="#PWR?"  Part="1"
-F 0 "#PWR?" H 5050 2550 50  0001 C CNN
+AR Path="/5C5EE841/5C5F2488" Ref="#PWR049"  Part="1"
+F 0 "#PWR049" H 5050 2550 50  0001 C CNN
 F 1 "GND" H 5055 2627 50  0000 C CNN
 F 2 "" H 5050 2800 50  0001 C CNN
@@
 P 6900 2500
 AR Path="/5C5F732E" Ref="Q?"  Part="1"
-AR Path="/5C5EE841/5C5F732E" Ref="Q?"  Part="1"
-F 0 "Q?" H 7150 2400 50  0000 C CNN
+AR Path="/5C5EE841/5C5F732E" Ref="Q3"  Part="1"
+F 0 "Q3" H 7150 2400 50  0000 C CNN
 F 1 "Q_NMOS_GDS" H 7350 2550 50  0000 C CNN
 F 2 "Package_TO_SOT_SMD:TO-252-2" H 7100 2600 50  0001 C CNN
@@
 P 6650 2150
 AR Path="/5C5F7335" Ref="D?"  Part="1"
-AR Path="/5C5EE841/5C5F7335" Ref="D?"  Part="1"
-F 0 "D?" H 6650 2350 50  0000 C CNN
+AR Path="/5C5EE841/5C5F7335" Ref="D5"  Part="1"
+F 0 "D5" H 6650 2350 50  0000 C CNN
 F 1 "1N4001" H 6650 2250 50  0000 C CNN
 F 2 "Diode_THT:D_DO-41_SOD81_P10.16mm_Horizontal" H 6650 2150 50  0001 C CNN
@@
 P 6450 2100
 AR Path="/5C5F733C" Ref="#PWR?"  Part="1"
-AR Path="/5C5EE841/5C5F733C" Ref="#PWR?"  Part="1"
-F 0 "#PWR?" H 6450 1950 50  0001 C CNN
+AR Path="/5C5EE841/5C5F733C" Ref="#PWR051"  Part="1"
+F 0 "#PWR051" H 6450 1950 50  0001 C CNN
 F 1 "+12V" H 6465 2273 50  0000 C CNN
 F 2 "" H 6450 2100 50  0001 C CNN
@@
 P 7400 2650
 AR Path="/5C5F7342" Ref="R?"  Part="1"
-AR Path="/5C5EE841/5C5F7342" Ref="R?"  Part="1"
-F 0 "R?" H 7332 2604 50  0000 R CNN
+AR Path="/5C5EE841/5C5F7342" Ref="R15"  Part="1"
+F 0 "R15" H 7332 2604 50  0000 R CNN
 F 1 "R_US" H 7332 2695 50  0000 R CNN
 F 2 "Resistor_SMD:R_0603_1608Metric" V 7440 2640 50  0001 C CNN
@@
 P 7250 2500
 AR Path="/5C5F7349" Ref="R?"  Part="1"
-AR Path="/5C5EE841/5C5F7349" Ref="R?"  Part="1"
-F 0 "R?" V 7150 2500 50  0000 C CNN
+AR Path="/5C5EE841/5C5F7349" Ref="R13"  Part="1"
+F 0 "R13" V 7150 2500 50  0000 C CNN
 F 1 "R_US" V 7350 2500 50  0000 C CNN
 F 2 "Resistor_SMD:R_0603_1608Metric" V 7290 2490 50  0001 C CNN
@@
 P 6800 2800
 AR Path="/5C5F7350" Ref="#PWR?"  Part="1"
-AR Path="/5C5EE841/5C5F7350" Ref="#PWR?"  Part="1"
-F 0 "#PWR?" H 6800 2550 50  0001 C CNN
+AR Path="/5C5EE841/5C5F7350" Ref="#PWR053"  Part="1"
+F 0 "#PWR053" H 6800 2550 50  0001 C CNN
 F 1 "GND" H 6805 2627 50  0000 C CNN
 F 2 "" H 6800 2800 50  0001 C CNN
@@
 P 7400 2800
 AR Path="/5C5F7357" Ref="#PWR?"  Part="1"
-AR Path="/5C5EE841/5C5F7357" Ref="#PWR?"  Part="1"
-F 0 "#PWR?" H 7400 2550 50  0001 C CNN
+AR Path="/5C5EE841/5C5F7357" Ref="#PWR055"  Part="1"
+F 0 "#PWR055" H 7400 2550 50  0001 C CNN
 F 1 "GND" H 7405 2627 50  0000 C CNN
 F 2 "" H 7400 2800 50  0001 C CNN
@@
 P 4550 4050
 AR Path="/5C5F7B5C" Ref="Q?"  Part="1"
-AR Path="/5C5EE841/5C5F7B5C" Ref="Q?"  Part="1"
-F 0 "Q?" H 4800 3950 50  0000 C CNN
+AR Path="/5C5EE841/5C5F7B5C" Ref="Q2"  Part="1"
+F 0 "Q2" H 4800 3950 50  0000 C CNN
 F 1 "Q_NMOS_GDS" H 5000 4100 50  0000 C CNN
 F 2 "Package_TO_SOT_SMD:TO-252-2" H 4750 4150 50  0001 C CNN
@@
 P 4300 3700
 AR Path="/5C5F7B63" Ref="D?"  Part="1"
-AR Path="/5C5EE841/5C5F7B63" Ref="D?"  Part="1"
-F 0 "D?" H 4300 3900 50  0000 C CNN
+AR Path="/5C5EE841/5C5F7B63" Ref="D4"  Part="1"
+F 0 "D4" H 4300 3900 50  0000 C CNN
 F 1 "1N4001" H 4300 3800 50  0000 C CNN
 F 2 "Diode_THT:D_DO-41_SOD81_P10.16mm_Horizontal" H 4300 3700 50  0001 C CNN
@@
 P 4100 3650
 AR Path="/5C5F7B6A" Ref="#PWR?"  Part="1"
-AR Path="/5C5EE841/5C5F7B6A" Ref="#PWR?"  Part="1"
-F 0 "#PWR?" H 4100 3500 50  0001 C CNN
+AR Path="/5C5EE841/5C5F7B6A" Ref="#PWR046"  Part="1"
+F 0 "#PWR046" H 4100 3500 50  0001 C CNN
 F 1 "+12V" H 4115 3823 50  0000 C CNN
 F 2 "" H 4100 3650 50  0001 C CNN
@@
 P 5050 4200
 AR Path="/5C5F7B70" Ref="R?"  Part="1"
-AR Path="/5C5EE841/5C5F7B70" Ref="R?"  Part="1"
-F 0 "R?" H 4982 4154 50  0000 R CNN
+AR Path="/5C5EE841/5C5F7B70" Ref="R12"  Part="1"
+F 0 "R12" H 4982 4154 50  0000 R CNN
 F 1 "R_US" H 4982 4245 50  0000 R CNN
 F 2 "Resistor_SMD:R_0603_1608Metric" V 5090 4190 50  0001 C CNN
@@
 P 4900 4050
 AR Path="/5C5F7B77" Ref="R?"  Part="1"
-AR Path="/5C5EE841/5C5F7B77" Ref="R?"  Part="1"
-F 0 "R?" V 4800 4050 50  0000 C CNN
+AR Path="/5C5EE841/5C5F7B77" Ref="R10"  Part="1"
+F 0 "R10" V 4800 4050 50  0000 C CNN
 F 1 "R_US" V 5000 4050 50  0000 C CNN
 F 2 "Resistor_SMD:R_0603_1608Metric" V 4940 4040 50  0001 C CNN
@@
 P 4450 4350
 AR Path="/5C5F7B7E" Ref="#PWR?"  Part="1"
-AR Path="/5C5EE841/5C5F7B7E" Ref="#PWR?"  Part="1"
-F 0 "#PWR?" H 4450 4100 50  0001 C CNN
+AR Path="/5C5EE841/5C5F7B7E" Ref="#PWR048"  Part="1"
+F 0 "#PWR048" H 4450 4100 50  0001 C CNN
 F 1 "GND" H 4455 4177 50  0000 C CNN
 F 2 "" H 4450 4350 50  0001 C CNN
@@
 P 5050 4350
 AR Path="/5C5F7B85" Ref="#PWR?"  Part="1"
-AR Path="/5C5EE841/5C5F7B85" Ref="#PWR?"  Part="1"
-F 0 "#PWR?" H 5050 4100 50  0001 C CNN
+AR Path="/5C5EE841/5C5F7B85" Ref="#PWR050"  Part="1"
+F 0 "#PWR050" H 5050 4100 50  0001 C CNN
 F 1 "GND" H 5055 4177 50  0000 C CNN
 F 2 "" H 5050 4350 50  0001 C CNN
@@
 P 6900 4050
 AR Path="/5C5F7B95" Ref="Q?"  Part="1"
-AR Path="/5C5EE841/5C5F7B95" Ref="Q?"  Part="1"
-F 0 "Q?" H 7150 3950 50  0000 C CNN
+AR Path="/5C5EE841/5C5F7B95" Ref="Q4"  Part="1"
+F 0 "Q4" H 7150 3950 50  0000 C CNN
 F 1 "Q_NMOS_GDS" H 7350 4100 50  0000 C CNN
 F 2 "Package_TO_SOT_SMD:TO-252-2" H 7100 4150 50  0001 C CNN
@@
 P 6650 3700
 AR Path="/5C5F7B9C" Ref="D?"  Part="1"
-AR Path="/5C5EE841/5C5F7B9C" Ref="D?"  Part="1"
-F 0 "D?" H 6650 3900 50  0000 C CNN
+AR Path="/5C5EE841/5C5F7B9C" Ref="D6"  Part="1"
+F 0 "D6" H 6650 3900 50  0000 C CNN
 F 1 "1N4001" H 6650 3800 50  0000 C CNN
 F 2 "Diode_THT:D_DO-41_SOD81_P10.16mm_Horizontal" H 6650 3700 50  0001 C CNN
@@
 P 6450 3650
 AR Path="/5C5F7BA3" Ref="#PWR?"  Part="1"
-AR Path="/5C5EE841/5C5F7BA3" Ref="#PWR?"  Part="1"
-F 0 "#PWR?" H 6450 3500 50  0001 C CNN
+AR Path="/5C5EE841/5C5F7BA3" Ref="#PWR052"  Part="1"
+F 0 "#PWR052" H 6450 3500 50  0001 C CNN
 F 1 "+12V" H 6465 3823 50  0000 C CNN
 F 2 "" H 6450 3650 50  0001 C CNN
@@
 P 7400 4200
 AR Path="/5C5F7BA9" Ref="R?"  Part="1"
-AR Path="/5C5EE841/5C5F7BA9" Ref="R?"  Part="1"
-F 0 "R?" H 7332 4154 50  0000 R CNN
+AR Path="/5C5EE841/5C5F7BA9" Ref="R16"  Part="1"
+F 0 "R16" H 7332 4154 50  0000 R CNN
 F 1 "R_US" H 7332 4245 50  0000 R CNN
 F 2 "Resistor_SMD:R_0603_1608Metric" V 7440 4190 50  0001 C CNN
@@
 P 7250 4050
 AR Path="/5C5F7BB0" Ref="R?"  Part="1"
-AR Path="/5C5EE841/5C5F7BB0" Ref="R?"  Part="1"
-F 0 "R?" V 7150 4050 50  0000 C CNN
+AR Path="/5C5EE841/5C5F7BB0" Ref="R14"  Part="1"
+F 0 "R14" V 7150 4050 50  0000 C CNN
 F 1 "R_US" V 7350 4050 50  0000 C CNN
 F 2 "Resistor_SMD:R_0603_1608Metric" V 7290 4040 50  0001 C CNN
@@
 P 6800 4350
 AR Path="/5C5F7BB7" Ref="#PWR?"  Part="1"
-AR Path="/5C5EE841/5C5F7BB7" Ref="#PWR?"  Part="1"
-F 0 "#PWR?" H 6800 4100 50  0001 C CNN
+AR Path="/5C5EE841/5C5F7BB7" Ref="#PWR054"  Part="1"
+F 0 "#PWR054" H 6800 4100 50  0001 C CNN
 F 1 "GND" H 6805 4177 50  0000 C CNN
 F 2 "" H 6800 4350 50  0001 C CNN
@@
 P 7400 4350
 AR Path="/5C5F7BBE" Ref="#PWR?"  Part="1"
-AR Path="/5C5EE841/5C5F7BBE" Ref="#PWR?"  Part="1"
-F 0 "#PWR?" H 7400 4100 50  0001 C CNN
+AR Path="/5C5EE841/5C5F7BBE" Ref="#PWR056"  Part="1"
+F 0 "#PWR056" H 7400 4100 50  0001 C CNN
 F 1 "GND" H 7405 4177 50  0000 C CNN
 F 2 "" H 7400 4350 50  0001 C CNN

Commit message: Getting there with layout of big board...
Parts:
- removed R10, R11, R12, R13, R14, R15, R16, R9: R_US, Resistor_SMD:R_0603_1608Metric, symbol Device:R_US
- added RN1: 1k, Resistor_SMD:R_Array_Convex_4x0603, symbol Device:R_Pack04
- added RN2: 10k, Resistor_SMD:R_Array_Convex_4x0603, symbol Device:R_Pack04
Connections:
- net FAN_CTRL_0: now also RN1.4 (R4.1), RN2.5 (R4.2)
- net FAN_CTRL_1: now also RN1.3 (R3.1), RN2.6 (R3.2)
- net FAN_CTRL_2: now also RN1.2 (R2.1), RN2.7 (R2.2)
- net FAN_CTRL_3: now also RN1.1 (R1.1), RN2.8 (R1.2)
- net GND: now also RN2.1 (R1.1), RN2.2 (R2.1), RN2.3 (R3.1), RN2.4 (R4.1)
- net at Q1.1 (G): now also RN1.5 (R4.2)
- net at Q3.1 (G): now also RN1.6 (R3.2)
- net at Q2.1 (G): now also RN1.7 (R2.2)
- net at Q4.1 (G): now also RN1.8 (R1.2)
Other:
- moved on the sheet: D3, D4, D5, D6, Q1, Q2, Q3, Q4
