File: interface-board/file5C667FAE.sch (KiCad schematic (older format))
At the start: 27 parts, among them U4 LTV-817S, U5 DCM4623TD2J13D0T70, U6 LTV-817S, U7 R-78E5.0-0.5, U9 TLP184

Commit message: Put Vicor on a removable module
Parts:
- removed C15, C17: 10uF, Capacitor_SMD:C_0603_1608Metric, symbol Device:C
- removed C16: 0.1uF, Capacitor_SMD:C_0603_1608Metric, symbol Device:C
- removed U7: R-78E5.0-0.5, Converter_DCDC:Converter_DCDC_RECOM_R-78E-0.5_THT, symbol Regulator_Switching:R-78E5.0-0.5
Other:
- note added: "Don't need this/doesn't work anyway (TRIM_HV is pulled up\ninternally, so should pull down through resistor/pot when \noptocoupler is on)"
- note added: "FAULT_HV can only supply 5mA absolute max, \nhence the different optocoupler choice."
- note added: "Will probably switch back to half\nas many 4700uF caps."
- note removed: "12V->5V"
Changed lines of the file:
@@
 $Descr A4 11693 8268
 encoding utf-8
-Sheet 4 5
+Sheet 4 6
 Title ""
 Date ""
@@
 Wire Wire Line
 	4350 3850 4800 3850
-$Comp
-L Regulator_Switching:R-78E5.0-0.5 U?
-U 1 1 5C66BF9B
-P 9000 3550
-AR Path="/5C66BF9B" Ref="U?"  Part="1"
-AR Path="/5C667FAF/5C66BF9B" Ref="U7"  Part="1"
-F 0 "U7" H 9000 3792 50  0000 C CNN
-F 1 "R-78E5.0-0.5" H 9000 3701 50  0000 C CNN
-F 2 "Converter_DCDC:Converter_DCDC_RECOM_R-78E-0.5_THT" H 9050 3300 50  0001 L CIN
-F 3 "https://www.recom-power.com/pdf/Innoline/R-78Exx-0.5.pdf" H 9000 3550 50  0001 C CNN
-	1    9000 3550
-	1    0    0    -1
-$EndComp
-Wire Wire Line
-	8550 3550 8700 3550
-Wire Wire Line
-	9450 3550 9300 3550
-$Comp
-L power:GND #PWR?
-U 1 1 5C66BFAA
-P 9000 3900
-AR Path="/5C66BFAA" Ref="#PWR?"  Part="1"
-AR Path="/5C667FAF/5C66BFAA" Ref="#PWR066"  Part="1"
-F 0 "#PWR066" H 9000 3650 50  0001 C CNN
-F 1 "GND" H 9005 3727 50  0000 C CNN
-F 2 "" H 9000 3900 50  0001 C CNN
-F 3 "" H 9000 3900 50  0001 C CNN
-	1    9000 3900
-	1    0    0    -1
-$EndComp
-Wire Wire Line
-	9000 3900 9000 3850
-Text Notes 8100 3050 0    100  ~ 0
-12V->5V
-$Comp
-L Device:C C?
-U 1 1 5C66BFB3
-P 9450 3700
-AR Path="/5C66BFB3" Ref="C?"  Part="1"
-AR Path="/5C667FAF/5C66BFB3" Ref="C16"  Part="1"
-F 0 "C16" H 9565 3746 50  0000 L CNN
-F 1 "0.1uF" H 9200 3600 50  0000 L CNN
-F 2 "Capacitor_SMD:C_0603_1608Metric" H 9488 3550 50  0001 C CNN
-F 3 "~" H 9450 3700 50  0001 C CNN
-	1    9450 3700
-	1    0    0    -1
-$EndComp
-Connection ~ 9450 3550
-$Comp
-L power:GND #PWR?
-U 1 1 5C66BFC5
-P 9600 3900
-AR Path="/5C66BFC5" Ref="#PWR?"  Part="1"
-AR Path="/5C667FAF/5C66BFC5" Ref="#PWR067"  Part="1"
-F 0 "#PWR067" H 9600 3650 50  0001 C CNN
-F 1 "GND" H 9605 3727 50  0000 C CNN
-F 2 "" H 9600 3900 50  0001 C CNN
-F 3 "" H 9600 3900 50  0001 C CNN
-	1    9600 3900
-	1    0    0    -1
-$EndComp
-Wire Wire Line
-	9450 3850 9600 3850
-Wire Wire Line
-	9600 3850 9600 3900
-Connection ~ 9600 3850
-Wire Wire Line
-	9600 3850 9750 3850
-$Comp
-L Device:C C?
-U 1 1 5C66BFCF
-P 8550 3700
-AR Path="/5C66BFCF" Ref="C?"  Part="1"
-AR Path="/5C667FAF/5C66BFCF" Ref="C15"  Part="1"
-F 0 "C15" H 8665 3746 50  0000 L CNN
-F 1 "10uF" H 8665 3655 50  0000 L CNN
-F 2 "Capacitor_SMD:C_0603_1608Metric" H 8588 3550 50  0001 C CNN
-F 3 "~" H 8550 3700 50  0001 C CNN
-	1    8550 3700
-	1    0    0    -1
-$EndComp
-$Comp
-L power:GND #PWR?
-U 1 1 5C66BFD7
-P 8550 3850
-AR Path="/5C66BFD7" Ref="#PWR?"  Part="1"
-AR Path="/5C667FAF/5C66BFD7" Ref="#PWR065"  Part="1"
-F 0 "#PWR065" H 8550 3600 50  0001 C CNN
-F 1 "GND" H 8555 3677 50  0000 C CNN
-F 2 "" H 8550 3850 50  0001 C CNN
-F 3 "" H 8550 3850 50  0001 C CNN
-	1    8550 3850
-	1    0    0    -1
-$EndComp
-Wire Notes Line
-	10150 2900 10150 4200
 Text HLabel 6200 1650 2    50   Input ~ 0
 TRIM_EN
@@
 Text HLabel 7200 5350 2    50   Input ~ 0
 12V_OUT
-Text HLabel 8500 3550 0    50   Input ~ 0
-12V_IN
-Wire Wire Line
-	8500 3550 8550 3550
-Connection ~ 8550 3550
-Wire Wire Line
-	9750 3550 9450 3550
-$Comp
-L Device:C C?
-U 1 1 5C66BFBA
-P 9750 3700
-AR Path="/5C66BFBA" Ref="C?"  Part="1"
-AR Path="/5C667FAF/5C66BFBA" Ref="C17"  Part="1"
-F 0 "C17" H 9865 3746 50  0000 L CNN
-F 1 "10uF" H 9865 3655 50  0000 L CNN
-F 2 "Capacitor_SMD:C_0603_1608Metric" H 9788 3550 50  0001 C CNN
-F 3 "~" H 9750 3700 50  0001 C CNN
-	1    9750 3700
-	1    0    0    -1
-$EndComp
-Text HLabel 9800 3550 2    50   Input ~ 0
-5V_OUT
-Wire Wire Line
-	9800 3550 9750 3550
-Connection ~ 9750 3550
 Wire Notes Line
 	3300 4650 7450 4650
@@
 Wire Notes Line
 	3350 6150 3350 5100
-Wire Notes Line
-	8050 4200 10150 4200
-Wire Notes Line
-	8050 2900 8050 4200
-Wire Notes Line
-	8050 2900 10150 2900
 Wire Notes Line width 39 rgb(253, 0, 0)
 	3150 1150 5400 1150
@@
 Wire Wire Line
 	6800 5350 7000 5350
+Text Notes 3500 2400 0    50   ~ 0
+Don't need this/doesn't work anyway (TRIM_HV is pulled up\ninternally, so should pull down through resistor/pot when \noptocoupler is on)
+Text Notes 5750 4100 0    50   ~ 0
+FAULT_HV can only supply 5mA absolute max, \nhence the different optocoupler choice.
+Text Notes 6050 6150 0    50   ~ 0
+Will probably switch back to half\nas many 4700uF caps.
 $EndSCHEMATC
