File: DC_DCBoard/TESTboard/_autosave-DC_DCBoard.kicad_pcb (KiCad board)
At the start: 2 copper layers, 137.2 x 68.6 mm, 31 parts, among them J1 TSV, J2 12V_OUT, J3 Conn_01x05, U1 DCM4623TD2J13D0T70, U2 LTV-817S, U3 TLP184, U4 LTV-817S

Commit message: Getting there with layout of big board...
Parts:
- F1: footprint Fuse:Fuseholder_Cylinder-5x20mm_Schurter_0031_8201_Horizontal_Open -> CustomFootprints:Fuseholder_Cylinder-5x20mm_Schurter_0031_8201_Horizontal_Open_3d
Changed lines of the file:
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@@
       (outputformat 1)
       (mirror false)
-      (drillshape 1)
+      (drillshape 0)
       (scaleselection 1)
-      (outputdirectory ""))
+      (outputdirectory "gerbers/"))
   )
   (net 0 "")
@@
     (add_net "Net-(C1-Pad1)")
     (add_net "Net-(F1-Pad1)")
+  )
+  (module CustomFootprints:Fuseholder_Cylinder-5x20mm_Schurter_0031_8201_Horizontal_Open_3d (layer F.Cu)
+    (at 81.28 118.745 90)
+    (descr http://www.schurter.com/var/schurter/storage/ilcatalogue/files/document/datasheet/en/pdf/typ_OGN.pdf)
+    (tags "Fuseholder horizontal open 5x20 Schurter 0031.8201")
+    (fp_text reference F1 (at -3.81 0 180) (layer F.SilkS)
+      (effects (font (size 1 1) (thickness 0.15)))
+    )
+    (fp_text value 2.5A (at 11.25 6 90) (layer F.Fab)
+      (effects (font (size 1 1) (thickness 0.15)))
+    )
+    (fp_text user %R (at 11.25 4 90) (layer F.Fab)
+      (effects (font (size 1 1) (thickness 0.15)))
+    )
+    (fp_line (start 0.1 -4.7) (end 0.1 4.7) (layer F.Fab) (width 0.1))
+    (fp_line (start 0.1 4.7) (end 22.4 4.7) (layer F.Fab) (width 0.1))
+    (fp_line (start 22.4 4.7) (end 22.4 -4.7) (layer F.Fab) (width 0.1))
+    (fp_line (start 22.4 -4.7) (end 0.1 -4.7) (layer F.Fab) (width 0.1))
+    (fp_line (start -0.25 5.05) (end -0.25 1.95) (layer F.CrtYd) (width 0.05))
+    (fp_line (start 22.5 4.8) (end 22.5 2) (layer F.SilkS) (width 0.12))
+    (fp_line (start 22.5 -2) (end 22.5 -4.8) (layer F.SilkS) (width 0.12))
+    (fp_line (start 0 -2) (end 0 -4.8) (layer F.SilkS) (width 0.12))
+    (fp_line (start 0 -4.8) (end 22.5 -4.8) (layer F.SilkS) (width 0.12))
+    (fp_line (start 22.75 5.05) (end -0.25 5.05) (layer F.CrtYd) (width 0.05))
+    (fp_line (start -0.25 -5.05) (end 22.75 -5.05) (layer F.CrtYd) (width 0.05))
+    (fp_line (start 0 4.8) (end 22.5 4.8) (layer F.SilkS) (width 0.12))
+    (fp_line (start -0.25 -1.95) (end -0.25 -5.05) (layer F.CrtYd) (width 0.05))
+    (fp_line (start 22.75 -1.95) (end 22.75 -5.05) (layer F.CrtYd) (width 0.05))
+    (fp_line (start 22.75 1.95) (end 22.75 5.05) (layer F.CrtYd) (width 0.05))
+    (fp_line (start 0 4.8) (end 0 2) (layer F.SilkS) (width 0.12))
+    (fp_arc (start 22.5 0) (end 22.75 -1.95) (angle 165.3) (layer F.CrtYd) (width 0.05))
+    (fp_arc (start 0 0) (end -0.25 1.95) (angle 165.3) (layer F.CrtYd) (width 0.05))
+    (pad 1 thru_hole circle (at 0 0 90) (size 3 3) (drill 1.3) (layers *.Cu *.Mask)
+      (net 7 "Net-(F1-Pad1)"))
+    (pad 2 thru_hole circle (at 22.5 0 90) (size 3 3) (drill 1.3) (layers *.Cu *.Mask)
+      (net 8 /HV+))
+    (pad "" np_thru_hole circle (at 11.25 0 90) (size 2.7 2.7) (drill 2.7) (layers *.Cu *.Mask))
+    (model ${KISYS3DMOD}/Fuse.3dshapes/Fuseholder_Cylinder-5x20mm_Schurter_0031_8201_Horizontal_Open.wrl
+      (at (xyz 0 0 0))
+      (scale (xyz 1 1 1))
+      (rotate (xyz 0 0 0))
+    )
+    (model "C:/Users/Willem Hillier/Documents/Github/AERO-boards-kicad/3d_models/31-8201.STEP"
+      (offset (xyz 11.4 0 0))
+      (scale (xyz 1 1 1))
+      (rotate (xyz -90 0 0))
+    )
   )
   (module CustomFootprints:DCM4623TD2J13D0T70_w_landpattern (layer F.Cu)
@@
       (at (xyz 0 0 0))
       (scale (xyz 1 1 1))
-      (rotate (xyz 0 0 0))
-    )
-  )
-  (module Fuse:Fuseholder_Cylinder-5x20mm_Schurter_0031_8201_Horizontal_Open (layer F.Cu)
-    (at 81.28 118.745 90)
-    (descr http://www.schurter.com/var/schurter/storage/ilcatalogue/files/document/datasheet/en/pdf/typ_OGN.pdf)
-    (tags "Fuseholder horizontal open 5x20 Schurter 0031.8201")
-    (fp_text reference F1 (at -3.81 0 180) (layer F.SilkS)
-      (effects (font (size 1 1) (thickness 0.15)))
-    )
-    (fp_text value 2.5A (at 11.25 6 90) (layer F.Fab)
-      (effects (font (size 1 1) (thickness 0.15)))
-    )
-    (fp_arc (start 0 0) (end -0.25 1.95) (angle 165.3) (layer F.CrtYd) (width 0.05))
-    (fp_arc (start 22.5 0) (end 22.75 -1.95) (angle 165.3) (layer F.CrtYd) (width 0.05))
-    (fp_line (start 0 4.8) (end 0 2) (layer F.SilkS) (width 0.12))
-    (fp_line (start 22.75 1.95) (end 22.75 5.05) (layer F.CrtYd) (width 0.05))
-    (fp_line (start 22.75 -1.95) (end 22.75 -5.05) (layer F.CrtYd) (width 0.05))
-    (fp_line (start -0.25 -1.95) (end -0.25 -5.05) (layer F.CrtYd) (width 0.05))
-    (fp_line (start 0 4.8) (end 22.5 4.8) (layer F.SilkS) (width 0.12))
-    (fp_line (start -0.25 -5.05) (end 22.75 -5.05) (layer F.CrtYd) (width 0.05))
-    (fp_line (start 22.75 5.05) (end -0.25 5.05) (layer F.CrtYd) (width 0.05))
-    (fp_line (start 0 -4.8) (end 22.5 -4.8) (layer F.SilkS) (width 0.12))
-    (fp_line (start 0 -2) (end 0 -4.8) (layer F.SilkS) (width 0.12))
-    (fp_line (start 22.5 -2) (end 22.5 -4.8) (layer F.SilkS) (width 0.12))
-    (fp_line (start 22.5 4.8) (end 22.5 2) (layer F.SilkS) (width 0.12))
-    (fp_line (start -0.25 5.05) (end -0.25 1.95) (layer F.CrtYd) (width 0.05))
-    (fp_line (start 22.4 -4.7) (end 0.1 -4.7) (layer F.Fab) (width 0.1))
-    (fp_line (start 22.4 4.7) (end 22.4 -4.7) (layer F.Fab) (width 0.1))
-    (fp_line (start 0.1 4.7) (end 22.4 4.7) (layer F.Fab) (width 0.1))
-    (fp_line (start 0.1 -4.7) (end 0.1 4.7) (layer F.Fab) (width 0.1))
-    (fp_text user %R (at 11.25 4 90) (layer F.Fab)
-      (effects (font (size 1 1) (thickness 0.15)))
-    )
-    (pad "" np_thru_hole circle (at 11.25 0 90) (size 2.7 2.7) (drill 2.7) (layers *.Cu *.Mask))
-    (pad 2 thru_hole circle (at 22.5 0 90) (size 3 3) (drill 1.3) (layers *.Cu *.Mask)
-      (net 8 /HV+))
-    (pad 1 thru_hole circle (at 0 0 90) (size 3 3) (drill 1.3) (layers *.Cu *.Mask)
-      (net 7 "Net-(F1-Pad1)"))
-    (model ${KISYS3DMOD}/Fuse.3dshapes/Fuseholder_Cylinder-5x20mm_Schurter_0031_8201_Horizontal_Open.wrl
-      (at (xyz 0 0 0))
-      (scale (xyz 1 1 1))
