File: interface-board-standoffs/file5C4BAF40.sch (KiCad schematic (older format))
At the start: 7 parts, among them U8 INA219

Commit message: Made rev1.1 of interface-board
Added i2c pullups, fixed chip pinout, added isolation slot, removed secondary DC/DC converter
Parts:
- added R10, R9: 10k, Resistor_SMD:R_0603_1608Metric, symbol Device:R_US
Connections:
- net +5V: now also R10.1, R9.1
- net SCL: now also R9.2
- net SDA: now also R10.2
Changed lines of the file:
@@
 Text Notes 8600 7050 0    100  ~ 0
 Willem Hillier\nUVM AERO\n3/5/2019
+$Comp
+L Device:R_US R9
+U 1 1 5CA4E022
+P 8400 3250
+F 0 "R9" H 8468 3296 50  0000 L CNN
+F 1 "10k" H 8468 3205 50  0000 L CNN
+F 2 "Resistor_SMD:R_0603_1608Metric" V 8440 3240 50  0001 C CNN
+F 3 "~" H 8400 3250 50  0001 C CNN
+	1    8400 3250
+	1    0    0    -1
+$EndComp
+$Comp
+L Device:R_US R10
+U 1 1 5CA4E102
+P 8750 3250
+F 0 "R10" H 8818 3296 50  0000 L CNN
+F 1 "10k" H 8818 3205 50  0000 L CNN
+F 2 "Resistor_SMD:R_0603_1608Metric" V 8790 3240 50  0001 C CNN
+F 3 "~" H 8750 3250 50  0001 C CNN
+	1    8750 3250
+	1    0    0    -1
+$EndComp
+Text HLabel 8400 3400 3    50   Input ~ 0
+SCL
+Text HLabel 8750 3400 3    50   Input ~ 0
+SDA
+$Comp
+L power:+5V #PWR0107
+U 1 1 5CA4E207
+P 8400 3100
+F 0 "#PWR0107" H 8400 2950 50  0001 C CNN
+F 1 "+5V" H 8415 3273 50  0000 C CNN
+F 2 "" H 8400 3100 50  0001 C CNN
+F 3 "" H 8400 3100 50  0001 C CNN
+	1    8400 3100
+	1    0    0    -1
+$EndComp
+$Comp
+L power:+5V #PWR0108
+U 1 1 5CA4E22B
+P 8750 3100
+F 0 "#PWR0108" H 8750 2950 50  0001 C CNN
+F 1 "+5V" H 8765 3273 50  0000 C CNN
+F 2 "" H 8750 3100 50  0001 C CNN
+F 3 "" H 8750 3100 50  0001 C CNN
+	1    8750 3100
+	1    0    0    -1
+$EndComp
 $EndSCHEMATC
