File: interface-board-standoffs/file5C83278D.sch (KiCad schematic (older format))
At the start: 19 parts, among them J1 HECS, J11 UART, J12 NTC1, J13 NTC1, J16 Conn_01x23, J2 CASEFAN1, J3 CASEFAN2, J4 Bender-LV, J5 BLINKY, J6 HV+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

Commit message: Made rev1.1 of interface-board
Added i2c pullups, fixed chip pinout, added isolation slot, removed secondary DC/DC converter
Parts:
- removed C1: 470uF, Capacitor_THT:CP_Radial_D10.0mm_P5.00mm, symbol Device:C
- removed J12, J13: NTC1, Connector_Molex:Molex_KK-254_AE-6410-02A_1x02_P2.54mm_Vertical, symbol Connector_Generic:Conn_01x02
- removed J2: CASEFAN1, Connector:FanPinHeader_1x03_P2.54mm_Vertical, symbol Connector_Generic:Conn_01x02
- removed J3: CASEFAN2, Connector:FanPinHeader_1x03_P2.54mm_Vertical, symbol Connector_Generic:Conn_01x02
- removed J5: BLINKY, Connector_Phoenix_MC_HighVoltage:PhoenixContact_MCV_1,5_2-G-5.08_1x02_P5.08mm_Vertical, symbol Connector_Generic:Conn_01x02
- removed U10: EPM1510SJ, CustomFootprints:EPM1510SJ, symbol interface-board-rescue:EPM1510SJ-CUSTOM_IC
- added J2: FANS, Connector_JST:JST_PH_B4B-PH-K_1x04_P2.00mm_Vertical, symbol Connector_Generic:Conn_01x04
- added J3: NTCs, Connector_JST:JST_PH_B4B-PH-K_1x04_P2.00mm_Vertical, symbol Connector_Generic:Conn_01x04
Connections:
- net labels added: HECS_AN1, HECS_AN2, HECS_AN3
- net labels removed: IMD_AN1, IMD_AN2, IMD_AN3
- wire segments 101 -> 97
Other:
- note removed: "Can remove this"
- note removed: "This is to run a HV indicator LED (called blinky)."
- moved on the sheet: J6, J7, J8
