File: interface-board-standoffs-biggerbox/file5C83278D.sch (KiCad schematic (older format))
At the start: 14 parts, among them J1 HECS, J11 UART, J16 Conn_01x23, J2 FANS, J3 NTCs, J4 Bender-LV, J6 HV+, J7 HV-, J8 HV+, U7 R-78E5.0-0.5

Commit message: Cleaned up drawings.user laser on interface-board, and made iBom for assembly.
Connections:
- net GND: now also J16.11 (Pin_11)
Changed lines of the file:
@@
 Wire Wire Line
 	1050 7450 1400 7450
+Wire Wire Line
+	1150 6450 1050 6450
 $EndSCHEMATC
