File: can-game-controller/can-game-controller.sch (KiCad schematic (older format))
At the start: 30 parts, among them J1 RJ45, J2 USB_B, J3 Pots, J4 Btns1, J5 Btns2, J6 Conn_02x03_Odd_Even, U1 MCP2551-I-SN, U2 MCP2515-xSO, U3 ATmega32U4-AU, Y1 8MHz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

Commit message: Finished USB CANBUS game controller
Will allow us to use the car as a game controller for a simulator
Parts:
- J6: footprint Connector_PinSocket_2.54mm:PinSocket_2x03_P2.54mm_Vertical -> Connector_PinHeader_2.54mm:PinHeader_2x03_P2.54mm_Vertical
Connections:
- net +5V: now also J3.2 (Pin_2), J3.5 (Pin_5); no longer J3.3 (Pin_3), J3.6 (Pin_6)
- net BTN2: now also U3.30 (PB6); no longer U3.31 (PC6)
- net BTN3: now also U3.28 (PB4); no longer U3.30 (PB6)
- net BTN4: now also U3.25 (PD4); no longer U3.29 (PB5)
- net BTN5: now also U3.31 (PC6); no longer U3.28 (PB4)
- net BTN6: now also U3.29 (PB5); no longer U3.27 (PD7)
- net BTN7: now also U3.27 (PD7); no longer U3.26 (PD6)
- net BTN8: now also U3.26 (PD6); no longer U3.25 (PD4)
- net GND: now also J3.7 (Pin_7); no longer J3.1 (Pin_1)
- net LED1: now also U3.18 (PD0)
- net LED2: now also U3.19 (PD1)
- net POT1: now also J3.6 (Pin_6); no longer J3.2 (Pin_2)
- net POT2: now also J3.3 (Pin_3); no longer J3.5 (Pin_5)
Other:
- moved on the sheet: J3
Changed lines of the file:
@@
 EESchema Schematic File Version 4
-LIBS:FanBoy-cache
+LIBS:can-game-controller-cache
 EELAYER 29 0
 EELAYER END
@@
 F 0 "J6" H 10450 1717 50  0000 C CNN
 F 1 "Conn_02x03_Odd_Even" H 10450 1626 50  0000 C CNN
-F 2 "Connector_PinSocket_2.54mm:PinSocket_2x03_P2.54mm_Vertical" H 10400 1400 50  0001 C CNN
+F 2 "Connector_PinHeader_2.54mm:PinHeader_2x03_P2.54mm_Vertical" H 10400 1400 50  0001 C CNN
 F 3 "~" H 10400 1400 50  0001 C CNN
 	1    10400 1400
@@
 Wire Wire Line
 	6250 1100 6250 1150
-Text Label 7200 1850 2    50   ~ 0
-BTN5
-Wire Wire Line
-	7200 1850 6950 1850
-Text Label 7200 1950 2    50   ~ 0
+Text Label 7200 3050 2    50   ~ 0
 BTN4
 Wire Wire Line
-	7200 1950 6950 1950
-Text Label 7200 2050 2    50   ~ 0
-BTN3
-Wire Wire Line
-	7200 2050 6950 2050
-Text Label 7200 2350 2    50   ~ 0
-BTN2
-Wire Wire Line
-	7200 2350 6950 2350
+	7200 3050 6950 3050
 Wire Wire Line
 	6950 2450 7200 2450
@@
 BTN1
 Wire Wire Line
+	7200 1950 6950 1950
+Text Label 7200 1950 2    50   ~ 0
+BTN6
+Wire Wire Line
 	7200 3350 6950 3350
 Text Label 7200 3350 2    50   ~ 0
-BTN6
-Wire Wire Line
-	7200 3250 6950 3250
-Text Label 7200 3250 2    50   ~ 0
 BTN7
-Wire Wire Line
-	7200 3050 6950 3050
-Text Label 7200 3050 2    50   ~ 0
-BTN8
 $Comp
 L power:GND #PWR0130
@@
 F 3 "~" H 10100 3250 50  0001 C CNN
 	1    10100 3250
-	1    0    0    -1
+	1    0    0    1
 $EndComp
 $Comp
@@
 Wire Wire Line
 	4850 1900 5200 1900
+Wire Wire Line
+	6950 2650 7200 2650
+Wire Wire Line
+	6950 2750 7200 2750
+Text Label 7200 2650 2    50   ~ 0
+LED1
+Text Label 7200 2750 2    50   ~ 0
+LED2
+Text Label 7200 2050 2    50   ~ 0
+BTN2
+Wire Wire Line
+	7200 2050 6950 2050
+Wire Wire Line
+	7200 2350 6950 2350
+Text Label 7200 2350 2    50   ~ 0
+BTN5
+Wire Wire Line
+	7200 1850 6950 1850
+Text Label 7200 1850 2    50   ~ 0
+BTN3
+Text Label 7200 3250 2    50   ~ 0
+BTN8
+Wire Wire Line
+	7200 3250 6950 3250
 $EndSCHEMATC
