File: TSAL-driver/TSAL-driver.sch (KiCad schematic (older format))
At the start: 28 parts, among them Q1 Q_PMOS_DGS, Q2 Q_NMOS_DGS, Q3 Q_NMOS_DGS, Q4 Q_NMOS_DGS, U1 LM556

Commit message: Added footprints for tsal-driver
Parts:
- C1: footprint (none) -> Capacitor_THT:CP_Radial_D6.3mm_P2.50mm
- C2, C3: footprint (none) -> Capacitor_SMD:C_0603_1608Metric
- C4, C5: footprint (none) -> Capacitor_SMD:C_0805_2012Metric_Pad1.15x1.40mm_HandSolder
- C6, C7: footprint (none) -> Capacitor_THT:C_Radial_D18.0mm_H35.5mm_P7.50mm
- C8: footprint (none) -> Capacitor_SMD:C_0805_2012Metric
- C9: footprint (none) -> Capacitor_SMD:C_0603_1608Metric_Pad1.05x0.95mm_HandSolder
- D1, D2: footprint (none) -> Diode_SMD:D_SMA
- J1, J2, J3, J4: renamed from J?; footprint (none) -> 1217861-1:TE_1217861-1
- Q1, Q2, Q3, Q4: footprint (none) -> Package_TO_SOT_SMD:TO-252-3_TabPin2
- R1, R2, R3, R4, R5, R6, R7: footprint (none) -> Resistor_SMD:R_0603_1608Metric
- R8: renamed from R?; footprint (none) -> Resistor_THT:R_Axial_Power_L48.0mm_W12.5mm_P60.96mm
- U1: footprint (none) -> Package_SO:SOIC-14_3.9x8.7mm_P1.27mm
Changed lines of the file:
@@
 F 0 "U1" H 1850 2250 50  0000 C CNN
 F 1 "LM556" H 2350 2250 50  0000 C CNN
-F 2 "" H 2100 1850 50  0001 C CNN
+F 2 "Package_SO:SOIC-14_3.9x8.7mm_P1.27mm" H 2100 1850 50  0001 C CNN
 F 3 "http://www.ti.com/lit/ds/symlink/lm556.pdf" H 2100 1850 50  0001 C CNN
 	1    2100 1850
@@
 F 0 "U1" H 5200 2250 50  0000 C CNN
 F 1 "LM556" H 5650 2250 50  0000 C CNN
-F 2 "" H 5450 1850 50  0001 C CNN
+F 2 "Package_SO:SOIC-14_3.9x8.7mm_P1.27mm" H 5450 1850 50  0001 C CNN
 F 3 "http://www.ti.com/lit/ds/symlink/lm556.pdf" H 5450 1850 50  0001 C CNN
 	2    5450 1850
@@
 F 0 "R4" V 3000 1850 50  0000 C CNN
 F 1 "100" V 3200 1850 50  0000 C CNN
-F 2 "" V 3140 1840 50  0001 C CNN
+F 2 "Resistor_SMD:R_0603_1608Metric" V 3140 1840 50  0001 C CNN
 F 3 "~" H 3100 1850 50  0001 C CNN
 	1    3100 1850
@@
 F 0 "C2" V 1400 1550 50  0000 C CNN
 F 1 "10n" V 1400 1800 50  0000 C CNN
-F 2 "" H 1350 1650 50  0001 C CNN
+F 2 "Capacitor_SMD:C_0603_1608Metric" H 1350 1650 50  0001 C CNN
 F 3 "~" H 1350 1650 50  0001 C CNN
 	1    1350 1650
@@
 F 0 "C3" V 1400 1750 50  0000 C CNN
 F 1 "0.01u" V 1400 2000 50  0000 C CNN
-F 2 "" H 1350 1850 50  0001 C CNN
+F 2 "Capacitor_SMD:C_0603_1608Metric" H 1350 1850 50  0001 C CNN
 F 3 "~" H 1350 1850 50  0001 C CNN
 	1    1350 1850
@@
 F 0 "R3" V 2800 2000 50  0000 C CNN
 F 1 "10k" V 2800 1750 50  0000 C CNN
-F 2 "" V 2790 1840 50  0001 C CNN
+F 2 "Resistor_SMD:R_0603_1608Metric" V 2790 1840 50  0001 C CNN
 F 3 "~" H 2750 1850 50  0001 C CNN
 	1    2750 1850
@@
 F 0 "R2" V 2700 1500 50  0000 C CNN
 F 1 "100" V 2700 1750 50  0000 C CNN
-F 2 "" V 2790 1640 50  0001 C CNN
+F 2 "Resistor_SMD:R_0603_1608Metric" V 2790 1640 50  0001 C CNN
 F 3 "~" H 2750 1650 50  0001 C CNN
 	1    2750 1650
@@
 F 0 "Q2" H 1606 3904 50  0000 L CNN
 F 1 "Q_NMOS_DGS" H 1606 3995 50  0000 L CNN
-F 2 "" H 1600 4050 50  0001 C CNN
+F 2 "Package_TO_SOT_SMD:TO-252-3_TabPin2" H 1600 4050 50  0001 C CNN
 F 3 "~" H 1400 3950 50  0001 C CNN
 	1    1400 3950
@@
 F 0 "Q1" H 1606 3596 50  0000 L CNN
 F 1 "Q_PMOS_DGS" H 1606 3505 50  0000 L CNN
-F 2 "" H 1600 3650 50  0001 C CNN
+F 2 "Package_TO_SOT_SMD:TO-252-3_TabPin2" H 1600 3650 50  0001 C CNN
 F 3 "~" H 1400 3550 50  0001 C CNN
 	1    1400 3550
@@
 F 0 "C1" H 1065 3296 50  0000 L CNN
 F 1 "100u" H 1065 3205 50  0000 L CNN
-F 2 "" H 988 3100 50  0001 C CNN
+F 2 "Capacitor_THT:CP_Radial_D6.3mm_P2.50mm" H 988 3100 50  0001 C CNN
 F 3 "~" H 950 3250 50  0001 C CNN
 	1    950  3250
@@
 F 0 "D1" H 1800 2995 50  0000 C CNN
 F 1 "1N4001" H 1800 3086 50  0000 C CNN
-F 2 "" V 1800 3200 50  0001 C CNN
+F 2 "Diode_SMD:D_SMA" V 1800 3200 50  0001 C CNN
 F 3 "~" V 1800 3200 50  0001 C CNN
 	1    1800 3200
@@
 F 0 "D2" H 2500 2995 50  0000 C CNN
 F 1 "1N4001" H 2500 3086 50  0000 C CNN
-F 2 "" V 2500 3200 50  0001 C CNN
+F 2 "Diode_SMD:D_SMA" V 2500 3200 50  0001 C CNN
 F 3 "~" V 2500 3200 50  0001 C CNN
 	1    2500 3200
@@
 F 0 "C4" H 2242 3496 50  0000 L CNN
 F 1 "10u" H 2242 3405 50  0000 L CNN
-F 2 "" H 2150 3450 50  0001 C CNN
+F 2 "Capacitor_SMD:C_0805_2012Metric_Pad1.15x1.40mm_HandSolder" H 2150 3450 50  0001 C CNN
 F 3 "~" H 2150 3450 50  0001 C CNN
 	1    2150 3450
@@
 F 0 "C5" H 2892 3496 50  0000 L CNN
 F 1 "10u" H 2892 3405 50  0000 L CNN
-F 2 "" H 2800 3450 50  0001 C CNN
+F 2 "Capacitor_SMD:C_0805_2012Metric_Pad1.15x1.40mm_HandSolder" H 2800 3450 50  0001 C CNN
 F 3 "~" H 2800 3450 50  0001 C CNN
 	1    2800 3450
@@
 F 0 "Q4" H 2406 5254 50  0000 L CNN
 F 1 "Q_NMOS_DGS" H 2406 5345 50  0000 L CNN
-F 2 "" H 2400 5400 50  0001 C CNN
+F 2 "Package_TO_SOT_SMD:TO-252-3_TabPin2" H 2400 5400 50  0001 C CNN
 F 3 "~" H 2200 5300 50  0001 C CNN
 	1    2200 5300
@@
 F 0 "R1" H 1868 5146 50  0000 L CNN
 F 1 "10k" H 1868 5055 50  0000 L CNN
-F 2 "" V 1840 5090 50  0001 C CNN
+F 2 "Resistor_SMD:R_0603_1608Metric" V 1840 5090 50  0001 C CNN
 F 3 "~" H 1800 5100 50  0001 C CNN
 	1    1800 5100
@@
 F 0 "Q3" H 1906 5454 50  0000 L CNN
 F 1 "Q_NMOS_DGS" H 1906 5545 50  0000 L CNN
-F 2 "" H 1900 5600 50  0001 C CNN
+F 2 "Package_TO_SOT_SMD:TO-252-3_TabPin2" H 1900 5600 50  0001 C CNN
 F 3 "~" H 1700 5500 50  0001 C CNN
 	1    1700 5500
@@
 F 0 "C6" H 3292 3396 50  0000 L CNN
 F 1 "4700uF" V 3100 3300 50  0000 L CNN
-F 2 "" H 3200 3350 50  0001 C CNN
+F 2 "Capacitor_THT:C_Radial_D18.0mm_H35.5mm_P7.50mm" H 3200 3350 50  0001 C CNN
 F 3 "~" H 3200 3350 50  0001 C CNN
 	1    3200 3350
@@
 F 0 "C7" H 3692 3396 50  0000 L CNN
 F 1 "4700uF" V 3500 3300 50  0000 L CNN
-F 2 "" H 3600 3350 50  0001 C CNN
+F 2 "Capacitor_THT:C_Radial_D18.0mm_H35.5mm_P7.50mm" H 3600 3350 50  0001 C CNN
 F 3 "~" H 3600 3350 50  0001 C CNN
 	1    3600 3350
@@
 F 0 "C8" V 4750 1550 50  0000 C CNN
 F 1 "10u" V 4750 1800 50  0000 C CNN
-F 2 "" H 4700 1650 50  0001 C CNN
+F 2 "Capacitor_SMD:C_0805_2012Metric" H 4700 1650 50  0001 C CNN
 F 3 "~" H 4700 1650 50  0001 C CNN
 	1    4700 1650
@@
 F 0 "C9" V 4750 1750 50  0000 C CNN
 F 1 "0.01" V 4750 2000 50  0000 C CNN
-F 2 "" H 4700 1850 50  0001 C CNN
+F 2 "Capacitor_SMD:C_0603_1608Metric_Pad1.05x0.95mm_HandSolder" H 4700 1850 50  0001 C CNN
 F 3 "~" H 4700 1850 50  0001 C CNN
 	1    4700 1850
@@
 F 0 "R7" V 6350 1850 50  0000 C CNN
 F 1 "39k" V 6550 1850 50  0000 C CNN
-F 2 "" V 6490 1840 50  0001 C CNN
+F 2 "Resistor_SMD:R_0603_1608Metric" V 6490 1840 50  0001 C CNN
 F 3 "~" H 6450 1850 50  0001 C CNN
 	1    6450 1850
@@
 F 0 "R6" V 6000 2000 50  0000 C CNN
 F 1 "4.7k" V 6000 1850 50  0000 C CNN
-F 2 "" V 6140 1840 50  0001 C CNN
+F 2 "Resistor_SMD:R_0603_1608Metric" V 6140 1840 50  0001 C CNN
 F 3 "~" H 6100 1850 50  0001 C CNN
 	1    6100 1850
@@
 F 0 "R5" V 5900 1650 50  0000 C CNN
 F 1 "100" V 6000 1650 50  0000 C CNN
-F 2 "" V 6140 1640 50  0001 C CNN
+F 2 "Resistor_SMD:R_0603_1608Metric" V 6140 1640 50  0001 C CNN
 F 3 "~" H 6100 1650 50  0001 C CNN
 	1    6100 1650
@@
 	9800 1550 9500 1550
 $Comp
-L Device:R_US R?
+L Device:R_US R8
 U 1 1 5D55FF69
 P 9500 2450
-F 0 "R?" V 9295 2450 50  0000 C CNN
+F 0 "R8" V 9295 2450 50  0000 C CNN
 F 1 "10" V 9386 2450 50  0000 C CNN
-F 2 "" V 9540 2440 50  0001 C CNN
+F 2 "Resistor_THT:R_Axial_Power_L48.0mm_W12.5mm_P60.96mm" V 9540 2440 50  0001 C CNN
 F 3 "~" H 9500 2450 50  0001 C CNN
 	1    9500 2450
@@
 	9650 2450 9750 2450
 $Comp
-L Connector:Screw_Terminal_01x01 J?
+L Connector:Screw_Terminal_01x01 J3
 U 1 1 5D64C9F5
 P 10000 1550
-F 0 "J?" H 9950 1650 50  0000 L CNN
+F 0 "J3" H 9950 1650 50  0000 L CNN
 F 1 "IN+" H 10050 1550 50  0000 L CNN
-F 2 "" H 10000 1550 50  0001 C CNN
+F 2 "1217861-1:TE_1217861-1" H 10000 1550 50  0001 C CNN
 F 3 "~" H 10000 1550 50  0001 C CNN
 	1    10000 1550
@@
 $EndComp
 $Comp
-L Connector:Screw_Terminal_01x01 J?
+L Connector:Screw_Terminal_01x01 J4
 U 1 1 5D64D107
 P 10000 1650
-F 0 "J?" H 9950 1550 50  0000 L CNN
+F 0 "J4" H 9950 1550 50  0000 L CNN
 F 1 "IN-" H 10050 1650 50  0000 L CNN
-F 2 "" H 10000 1650 50  0001 C CNN
+F 2 "1217861-1:TE_1217861-1" H 10000 1650 50  0001 C CNN
 F 3 "~" H 10000 1650 50  0001 C CNN
 	1    10000 1650
@@
 	10250 950  10250 2700
 $Comp
-L Connector:Screw_Terminal_01x01 J?
+L Connector:Screw_Terminal_01x01 J1
 U 1 1 5D65087F
 P 9950 2450
-F 0 "J?" H 9900 2550 50  0000 L CNN
+F 0 "J1" H 9900 2550 50  0000 L CNN
 F 1 "OUT+" H 10000 2450 50  0000 L CNN
-F 2 "" H 9950 2450 50  0001 C CNN
+F 2 "1217861-1:TE_1217861-1" H 9950 2450 50  0001 C CNN
 F 3 "~" H 9950 2450 50  0001 C CNN
 	1    9950 2450
@@
 $EndComp
 $Comp
-L Connector:Screw_Terminal_01x01 J?
+L Connector:Screw_Terminal_01x01 J2
 U 1 1 5D650885
 P 9950 2550
-F 0 "J?" H 9900 2450 50  0000 L CNN
+F 0 "J2" H 9900 2450 50  0000 L CNN
 F 1 "OUT-" H 10000 2550 50  0000 L CNN
-F 2 "" H 9950 2550 50  0001 C CNN
+F 2 "1217861-1:TE_1217861-1" H 9950 2550 50  0001 C CNN
 F 3 "~" H 9950 2550 50  0001 C CNN
 	1    9950 2550

Commit message: New TSAL Schematic
Schematic complete, on to annotations
Parts:
- removed C1: 100u, Capacitor_THT:CP_Radial_D6.3mm_P2.50mm, symbol Device:C
- removed C6, C7: 4700uF, Capacitor_THT:C_Radial_D18.0mm_H35.5mm_P7.50mm, symbol Device:C_Small
- removed C8: 10u, Capacitor_SMD:C_0805_2012Metric, symbol Device:C_Small
- removed C9: 0.01, Capacitor_SMD:C_0603_1608Metric_Pad1.05x0.95mm_HandSolder, symbol Device:C_Small
- removed D1, D2: 1N4001, Diode_SMD:D_SMA, symbol Device:D_Small
- removed J1: OUT+, 1217861-1:TE_1217861-1, symbol Connector:Screw_Terminal_01x01
- removed J2: OUT-, 1217861-1:TE_1217861-1, symbol Connector:Screw_Terminal_01x01
- removed J3: IN+, 1217861-1:TE_1217861-1, symbol Connector:Screw_Terminal_01x01
- removed J4: IN-, 1217861-1:TE_1217861-1, symbol Connector:Screw_Terminal_01x01
- removed Q1: Q_PMOS_DGS, Package_TO_SOT_SMD:TO-252-3_TabPin2, symbol Device:Q_PMOS_DGS
- removed Q2, Q3, Q4: Q_NMOS_DGS, Package_TO_SOT_SMD:TO-252-3_TabPin2, symbol Device:Q_NMOS_DGS
- removed R1, R3: 10k, Resistor_SMD:R_0603_1608Metric, symbol Device:R_US
- removed R2, R4, R5: 100, Resistor_SMD:R_0603_1608Metric, symbol Device:R_US
- removed R6: 4.7k, Resistor_SMD:R_0603_1608Metric, symbol Device:R_US
- removed R7: 39k, Resistor_SMD:R_0603_1608Metric, symbol Device:R_US
- removed R8: 10, Resistor_THT:R_Axial_Power_L48.0mm_W12.5mm_P60.96mm, symbol Device:R_US
- removed U1: LM556, Package_SO:SOIC-14_3.9x8.7mm_P1.27mm, symbol Timer:LM556
- added +Vin1: 12V, symbol Connector_Generic:Conn_01x01
- added +Vout1: LED+, symbol Connector_Generic:Conn_01x01
- added -Vin1: GND, symbol Connector_Generic:Conn_01x01
- added -Vout1: LED-, symbol Connector_Generic:Conn_01x01
- added C1: 0.1uF, symbol Device:C_Small
- added U1: R-78E5.0-0.5, Converter_DCDC:Converter_DCDC_RECOM_R-78E-0.5_THT, symbol Regulator_Switching:R-78E5.0-0.5
- added U2: ATtiny25-20SU, Package_SO:SOIJ-8_5.3x5.3mm_P1.27mm, symbol MCU_Microchip_ATtiny:ATtiny25-20SU
- added U3: LDB-350L, symbol AERO_custom_symbols:LDB-350L
- C2: value 10n -> 10uF; footprint Capacitor_SMD:C_0603_1608Metric -> (none)
- C3: value 0.01u -> 10uF; footprint Capacitor_SMD:C_0603_1608Metric -> (none)
- C4, C5: value 10u -> 10uF; footprint Capacitor_SMD:C_0805_2012Metric_Pad1.15x1.40mm_HandSolder -> (none)
Connections:
- net labels added: +5V, PWM_DIM
- net labels removed: BLINK_PWM_INVERTED, LED-, VDOUBLE_PWM
- wire segments 57 -> 20
Other:
- note added: "12V -> 24V DC/DC"
- note added: "12V -> 5V DC/DC"
- note added: "Connectors\n"
- note added: "uC"
- note removed: "BLINKER"
- note removed: "CONNECTORS"
- note removed: "LED DRIVER"
- note removed: "VOLTAGE DOUBLER"

Commit message: started choosing footprints
Parts:
- C1, C2, C3, C4, C5: footprint (none) -> Capacitor_SMD:C_0603_1608Metric
Changed lines of the file:
@@
 F 0 "C4" H 5808 4154 50  0000 R CNN
 F 1 "10uF" H 5808 4245 50  0000 R CNN
-F 2 "" H 5900 4200 50  0001 C CNN
+F 2 "Capacitor_SMD:C_0603_1608Metric" H 5900 4200 50  0001 C CNN
 F 3 "~" H 5900 4200 50  0001 C CNN
 	1    5900 4200
@@
 F 0 "C5" H 6208 4154 50  0000 R CNN
 F 1 "10uF" H 6208 4245 50  0000 R CNN
-F 2 "" H 6300 4200 50  0001 C CNN
+F 2 "Capacitor_SMD:C_0603_1608Metric" H 6300 4200 50  0001 C CNN
 F 3 "~" H 6300 4200 50  0001 C CNN
 	1    6300 4200
@@
 F 0 "C2" H 2958 5154 50  0000 R CNN
 F 1 "10uF" H 2958 5245 50  0000 R CNN
-F 2 "" H 3050 5200 50  0001 C CNN
+F 2 "Capacitor_SMD:C_0603_1608Metric" H 3050 5200 50  0001 C CNN
 F 3 "~" H 3050 5200 50  0001 C CNN
 	1    3050 5200
@@
 F 0 "C3" H 4058 5154 50  0000 R CNN
 F 1 "10uF" H 4058 5245 50  0000 R CNN
-F 2 "" H 4150 5200 50  0001 C CNN
+F 2 "Capacitor_SMD:C_0603_1608Metric" H 4150 5200 50  0001 C CNN
 F 3 "~" H 4150 5200 50  0001 C CNN
 	1    4150 5200
@@
 F 0 "C1" H 2842 3196 50  0000 L CNN
 F 1 "0.1uF" H 2850 3100 50  0000 L CNN
-F 2 "" H 2750 3150 50  0001 C CNN
+F 2 "Capacitor_SMD:C_0603_1608Metric" H 2750 3150 50  0001 C CNN
 F 3 "~" H 2750 3150 50  0001 C CNN
 	1    2750 3150

Commit message: Finished TSAL-driver
Parts:
- removed C5: 10uF, Capacitor_SMD:C_0603_1608Metric, symbol Device:C_Small
- removed U1: R-78E5.0-0.5, Converter_DCDC:Converter_DCDC_RECOM_R-78E-0.5_THT, symbol Regulator_Switching:R-78E5.0-0.5
- removed U2: ATtiny25-20SU, Package_SO:SOIJ-8_5.3x5.3mm_P1.27mm, symbol MCU_Microchip_ATtiny:ATtiny25-20SU
- added U1: AZ1117-5.0, Package_TO_SOT_SMD:SOT-223-3_TabPin2, symbol Regulator_Linear:AZ1117-5.0
- added U2: ATtiny25-20SSU, Package_SO:SOIC-8_3.9x4.9mm_P1.27mm, symbol MCU_Microchip_ATtiny:ATtiny25-20SSU
- J1: renamed from +Vout1; footprint (none) -> AERO-footprints:TE_1217861-1
- J2: renamed from -Vout1; footprint (none) -> AERO-footprints:TE_1217861-1
- J3: renamed from +Vin1; footprint (none) -> AERO-footprints:TE_1217861-1
- J4: renamed from -Vin1; footprint (none) -> AERO-footprints:TE_1217861-1
- U3: footprint (none) -> AERO-footprints:DIP1549W45P254L3404H940Q24
Connections:
- net +12V: now also C2.2, U1.3 (VI)
- net +24V: no longer C2.2
- net +5V: now also U1.2 (VO), U2.8 (VCC)
- net GND: now also U1.1 (GND), U2.4 (GND)
- net PWM_DIM: now also U2.6 (PB1)
Other:
- moved on the sheet: C4
Changed lines of the file:
@@
 F 0 "U3" H 6100 3765 50  0000 C CNN
 F 1 "LDB-350L" H 6100 3674 50  0000 C CNN
-F 2 "" H 6250 3200 50  0001 C CNN
+F 2 "AERO-footprints:DIP1549W45P254L3404H940Q24" H 6250 3200 50  0001 C CNN
 F 3 "" H 6250 3200 50  0001 C CNN
 	1    6100 3150
@@
 L Device:C_Small C4
 U 1 1 5D9E14E9
-P 5900 4200
-F 0 "C4" H 5808 4154 50  0000 R CNN
-F 1 "10uF" H 5808 4245 50  0000 R CNN
-F 2 "Capacitor_SMD:C_0603_1608Metric" H 5900 4200 50  0001 C CNN
-F 3 "~" H 5900 4200 50  0001 C CNN
-	1    5900 4200
+P 6050 4200
+F 0 "C4" H 5958 4154 50  0000 R CNN
+F 1 "10uF" H 5958 4245 50  0000 R CNN
+F 2 "Capacitor_SMD:C_0603_1608Metric" H 6050 4200 50  0001 C CNN
+F 3 "~" H 6050 4200 50  0001 C CNN
+	1    6050 4200
 	-1   0    0    1
 $EndComp
@@
 L power:GND #PWR0104
 U 1 1 5D9E14EF
-P 5900 4400
-F 0 "#PWR0104" H 5900 4150 50  0001 C CNN
-F 1 "GND" H 5905 4227 50  0000 C CNN
-F 2 "" H 5900 4400 50  0001 C CNN
-F 3 "" H 5900 4400 50  0001 C CNN
-	1    5900 4400
-	1    0    0    -1
-$EndComp
-Wire Wire Line
-	5900 4300 5900 4400
+P 6050 4400
+F 0 "#PWR0104" H 6050 4150 50  0001 C CNN
+F 1 "GND" H 6055 4227 50  0000 C CNN
+F 2 "" H 6050 4400 50  0001 C CNN
+F 3 "" H 6050 4400 50  0001 C CNN
+	1    6050 4400
+	1    0    0    -1
+$EndComp
+Wire Wire Line
+	6050 4300 6050 4400
 Wire Wire Line
 	6600 3300 6700 3300
@@
 L power:+12V #PWR0106
 U 1 1 5D9EBE4E
-P 5900 4100
-F 0 "#PWR0106" H 5900 3950 50  0001 C CNN
-F 1 "+12V" V 5915 4228 50  0000 L CNN
-F 2 "" H 5900 4100 50  0001 C CNN
-F 3 "" H 5900 4100 50  0001 C CNN
-	1    5900 4100
-	1    0    0    -1
-$EndComp
-$Comp
-L Device:C_Small C5
-U 1 1 5D9EDDD0
-P 6300 4200
-F 0 "C5" H 6208 4154 50  0000 R CNN
-F 1 "10uF" H 6208 4245 50  0000 R CNN
-F 2 "Capacitor_SMD:C_0603_1608Metric" H 6300 4200 50  0001 C CNN
-F 3 "~" H 6300 4200 50  0001 C CNN
-	1    6300 4200
-	-1   0    0    1
-$EndComp
-$Comp
-L power:GND #PWR0107
-U 1 1 5D9EDDD6
-P 6300 4400
-F 0 "#PWR0107" H 6300 4150 50  0001 C CNN
-F 1 "GND" H 6305 4227 50  0000 C CNN
-F 2 "" H 6300 4400 50  0001 C CNN
-F 3 "" H 6300 4400 50  0001 C CNN
-	1    6300 4400
-	1    0    0    -1
-$EndComp
-Wire Wire Line
-	6300 4300 6300 4400
-$Comp
-L power:+24V #PWR0108
-U 1 1 5D9EEAE3
-P 6300 4100
-F 0 "#PWR0108" H 6300 3950 50  0001 C CNN
-F 1 "+24V" V 6315 4228 50  0000 L CNN
-F 2 "" H 6300 4100 50  0001 C CNN
-F 3 "" H 6300 4100 50  0001 C CNN
-	1    6300 4100
+P 6050 4100
+F 0 "#PWR0106" H 6050 3950 50  0001 C CNN
+F 1 "+12V" V 6065 4228 50  0000 L CNN
+F 2 "" H 6050 4100 50  0001 C CNN
+F 3 "" H 6050 4100 50  0001 C CNN
+	1    6050 4100
 	1    0    0    -1
 $EndComp
@@
 $EndComp
 $Comp
-L Connector_Generic:Conn_01x01 -Vin1
+L Connector_Generic:Conn_01x01 J4
 U 1 1 5D9B7D4E
 P 8350 3650
-F 0 "-Vin1" H 8430 3692 50  0000 L CNN
+F 0 "J4" H 8430 3692 50  0000 L CNN
 F 1 "GND" H 8430 3601 50  0000 L CNN
-F 2 "" H 8350 3650 50  0001 C CNN
+F 2 "AERO-footprints:TE_1217861-1" H 8350 3650 50  0001 C CNN
 F 3 "~" H 8350 3650 50  0001 C CNN
 	1    8350 3650
@@
 $EndComp
 $Comp
-L Connector_Generic:Conn_01x01 +Vin1
+L Connector_Generic:Conn_01x01 J3
 U 1 1 5D9B7803
 P 8350 3450
-F 0 "+Vin1" H 8430 3492 50  0000 L CNN
+F 0 "J3" H 8430 3492 50  0000 L CNN
 F 1 "12V" H 8430 3401 50  0000 L CNN
-F 2 "" H 8350 3450 50  0001 C CNN
+F 2 "AERO-footprints:TE_1217861-1" H 8350 3450 50  0001 C CNN
 F 3 "~" H 8350 3450 50  0001 C CNN
 	1    8350 3450
@@
 $EndComp
 $Comp
-L Connector_Generic:Conn_01x01 -Vout1
+L Connector_Generic:Conn_01x01 J2
 U 1 1 5D9B716F
 P 8350 3250
-F 0 "-Vout1" H 8430 3292 50  0000 L CNN
+F 0 "J2" H 8430 3292 50  0000 L CNN
 F 1 "LED-" H 8430 3201 50  0000 L CNN
-F 2 "" H 8350 3250 50  0001 C CNN
+F 2 "AERO-footprints:TE_1217861-1" H 8350 3250 50  0001 C CNN
 F 3 "~" H 8350 3250 50  0001 C CNN
 	1    8350 3250
@@
 $EndComp
 $Comp
-L Connector_Generic:Conn_01x01 +Vout1
+L Connector_Generic:Conn_01x01 J1
 U 1 1 5D9B58C1
 P 8350 3050
-F 0 "+Vout1" H 8430 3092 50  0000 L CNN
+F 0 "J1" H 8430 3092 50  0000 L CNN
 F 1 "LED+" H 8430 3001 50  0000 L CNN
-F 2 "" H 8350 3050 50  0001 C CNN
+F 2 "AERO-footprints:TE_1217861-1" H 8350 3050 50  0001 C CNN
 F 3 "~" H 8350 3050 50  0001 C CNN
 	1    8350 3050
@@
 F 3 "" H 4150 5050 50  0001 C CNN
 	1    4150 5050
-	1    0    0    -1
-$EndComp
-$Comp
-L power:+24V #PWR0117
-U 1 1 5D99D790
-P 3050 5050
-F 0 "#PWR0117" H 3050 4900 50  0001 C CNN
-F 1 "+24V" V 3065 5178 50  0000 L CNN
-F 2 "" H 3050 5050 50  0001 C CNN
-F 3 "" H 3050 5050 50  0001 C CNN
-	1    3050 5050
-	1    0    0    -1
-$EndComp
-$Comp
-L power:+24V #PWR0118
-U 1 1 5D98475D
-P 3250 5050
-F 0 "#PWR0118" H 3250 4900 50  0001 C CNN
-F 1 "+24V" V 3265 5178 50  0000 L CNN
-F 2 "" H 3250 5050 50  0001 C CNN
-F 3 "" H 3250 5050 50  0001 C CNN
-	1    3250 5050
 	1    0    0    -1
 $EndComp
@@
 $EndComp
 Wire Wire Line
-	4600 2950 4250 2950
+	4600 2950 4300 2950
 Text Label 4600 2950 2    50   ~ 0
 PWM_DIM
@@
 Text Notes 3550 2200 0    100  ~ 20
 uC
-$Comp
-L MCU_Microchip_ATtiny:ATtiny25-20SU U2
-U 1 1 5D978C35
-P 3650 3150
-F 0 "U2" H 3850 3750 50  0000 R CNN
-F 1 "ATtiny25-20SU" H 3500 3750 50  0000 R CNN
-F 2 "Package_SO:SOIJ-8_5.3x5.3mm_P1.27mm" H 3650 3150 50  0001 C CIN
-F 3 "http://ww1.microchip.com/downloads/en/DeviceDoc/atmel-2586-avr-8-bit-microcontroller-attiny25-attiny45-attiny85_datasheet.pdf" H 3650 3150 50  0001 C CNN
-	1    3650 3150
-	1    0    0    -1
-$EndComp
-$Comp
-L Regulator_Switching:R-78E5.0-0.5 U1
-U 1 1 5D97F1B0
-P 3600 5100
-F 0 "U1" H 3600 5342 50  0000 C CNN
-F 1 "R-78E5.0-0.5" H 3600 5251 50  0000 C CNN
-F 2 "Converter_DCDC:Converter_DCDC_RECOM_R-78E-0.5_THT" H 3650 4850 50  0001 L CIN
-F 3 "https://www.recom-power.com/pdf/Innoline/R-78Exx-0.5.pdf" H 3600 5100 50  0001 C CNN
-	1    3600 5100
-	1    0    0    -1
-$EndComp
 $Comp
 L power:GND #PWR0119
@@
 	7150 1950 7150 4900
 $Comp
+L power:GND #PWR0122
+U 1 1 5DA4A45C
+P 2750 3250
+F 0 "#PWR0122" H 2750 3000 50  0001 C CNN
+F 1 "GND" H 2755 3077 50  0000 C CNN
+F 2 "" H 2750 3250 50  0001 C CNN
+F 3 "" H 2750 3250 50  0001 C CNN
+	1    2750 3250
+	1    0    0    -1
+$EndComp
+$Comp
+L power:+5V #PWR0123
+U 1 1 5DA4A891
+P 2750 3050
+F 0 "#PWR0123" H 2750 2900 50  0001 C CNN
+F 1 "+5V" H 2765 3223 50  0000 C CNN
+F 2 "" H 2750 3050 50  0001 C CNN
+F 3 "" H 2750 3050 50  0001 C CNN
+	1    2750 3050
+	1    0    0    -1
+$EndComp
+$Comp
+L MCU_Microchip_ATtiny:ATtiny25-20SSU U2
+U 1 1 5D9E8B2B
+P 3650 3150
+F 0 "U2" H 3900 3700 50  0000 R CNN
+F 1 "ATtiny25-20SSU" H 4400 3800 50  0000 R CNN
+F 2 "Package_SO:SOIC-8_3.9x4.9mm_P1.27mm" H 3650 3150 50  0001 C CIN
+F 3 "http://ww1.microchip.com/downloads/en/DeviceDoc/atmel-2586-avr-8-bit-microcontroller-attiny25-attiny45-attiny85_datasheet.pdf" H 3650 3150 50  0001 C CNN
+	1    3650 3150
+	1    0    0    -1
+$EndComp
+Connection ~ 4300 2950
+Wire Wire Line
+	4300 2950 4250 2950
+$Comp
 L Device:C_Small C1
 U 1 1 5DA46C87
@@
 $EndComp
 $Comp
-L power:GND #PWR0122
-U 1 1 5DA4A45C
-P 2750 3250
-F 0 "#PWR0122" H 2750 3000 50  0001 C CNN
-F 1 "GND" H 2755 3077 50  0000 C CNN
-F 2 "" H 2750 3250 50  0001 C CNN
-F 3 "" H 2750 3250 50  0001 C CNN
-	1    2750 3250
-	1    0    0    -1
-$EndComp
-$Comp
-L power:+5V #PWR0123
-U 1 1 5DA4A891
-P 2750 3050
-F 0 "#PWR0123" H 2750 2900 50  0001 C CNN
-F 1 "+5V" H 2765 3223 50  0000 C CNN
-F 2 "" H 2750 3050 50  0001 C CNN
-F 3 "" H 2750 3050 50  0001 C CNN
-	1    2750 3050
-	1    0    0    -1
-$EndComp
+L Regulator_Linear:AZ1117-5.0 U1
+U 1 1 5D9EE5E1
+P 3600 5100
+F 0 "U1" H 3600 5342 50  0000 C CNN
+F 1 "AZ1117-5.0" H 3600 5251 50  0000 C CNN
+F 2 "Package_TO_SOT_SMD:SOT-223-3_TabPin2" H 3600 5350 50  0001 C CIN
+F 3 "https://www.diodes.com/assets/Datasheets/AZ1117.pdf" H 3600 5100 50  0001 C CNN
+	1    3600 5100
+	1    0    0    -1
+$EndComp
+$Comp
+L power:+12V #PWR0107
+U 1 1 5D9F1D60
+P 3050 5050
+F 0 "#PWR0107" H 3050 4900 50  0001 C CNN
+F 1 "+12V" H 3065 5223 50  0000 C CNN
+F 2 "" H 3050 5050 50  0001 C CNN
+F 3 "" H 3050 5050 50  0001 C CNN
+	1    3050 5050
+	1    0    0    -1
+$EndComp
+$Comp
+L power:+12V #PWR0108
+U 1 1 5D9F1F75
+P 3250 5050
+F 0 "#PWR0108" H 3250 4900 50  0001 C CNN
+F 1 "+12V" H 3265 5223 50  0000 C CNN
+F 2 "" H 3250 5050 50  0001 C CNN
+F 3 "" H 3250 5050 50  0001 C CNN
+	1    3250 5050
+	1    0    0    -1
+$EndComp
