File: demo-board/demo-board.sch (KiCad schematic (older format))
At the start: 22 parts

Commit message: Demo Board updated. Ready for Review
Parts:
- removed C?: 0.1u, symbol Device:C_Small
- removed C?: 10u, symbol Device:C_Small
- removed D? (x8): WS2812B, LED_SMD:LED_WS2812B_PLCC4_5.0x5.0mm_P3.2mm, symbol LED:WS2812B
- removed J?: USB_B_Micro, symbol Connector:USB_B_Micro
- removed J?: Conn_02x03_Odd_Even, symbol Connector_Generic:Conn_02x03_Odd_Even
- removed JP? (x8): Jumper_2_Open, symbol Jumper:Jumper_2_Open
- removed R?: 10k, symbol Device:R_US
- removed U?: ATtiny85-20SU, Package_SO:SOIJ-8_5.3x5.3mm_P1.27mm, symbol MCU_Microchip_ATtiny:ATtiny85-20SU
- added C1: 0.1U, Capacitor_SMD:C_0603_1608Metric_Pad1.05x0.95mm_HandSolder, symbol Device:C
- added C2: 10U, Capacitor_SMD:C_0603_1608Metric_Pad1.05x0.95mm_HandSolder, symbol Device:C
- added D1, D2, D3, D4, D5, D6, D7, D8: WS2812B, LED_SMD:LED_WS2812B_PLCC4_5.0x5.0mm_P3.2mm, symbol LED:WS2812B
- added J1: USB_B_Micro, Connector_USB:USB_Micro-B_Molex-105017-0001, symbol Connector:USB_B_Micro
- added J2: Conn_02x03_Odd_Even, Connector_PinHeader_2.54mm:PinHeader_2x03_P2.54mm_Vertical, symbol Connector_Generic:Conn_02x03_Odd_Even
- added JP1, JP2, JP3, JP4, JP5, JP6, JP7, JP8: Jumper_2_Open, Jumper:SolderJumper-2_P1.3mm_Open_RoundedPad1.0x1.5mm, symbol Jumper:Jumper_2_Open
- added R1: 1OK, Resistor_SMD:R_0603_1608Metric_Pad1.05x0.95mm_HandSolder, symbol Device:R
- added U1: ATtiny85-20SU, Package_SO:SOIJ-8_5.3x5.3mm_P1.27mm, symbol MCU_Microchip_ATtiny:ATtiny85-20SU
Connections:
- wire segments 64 -> 61
